File: Power.kicad_sch (KiCad schematic)
At the start: 67 parts, among them Q1 FDMC86240, Q2 FDMC86240, U1 LM5155DSSR, U2 LM5155DSSR, U8 TPS51385RJNR

Commit message: almost finished, phew! just dd +/- 5v rails, connect the SDIO & power enable pins and figure out the rest of the clocking chain
Parts:
- removed C14, C195, C196, C60: 10uF, symbol Device:C
- removed C193, C206: 47nF, symbol Device:C
- removed C194, C197: 100nF, symbol Device:C
- removed C199: 300nF, symbol Device:C
- removed C200, C201: 2.2uF, symbol Device:C
- removed C202, C203, C204, C205, C55, C56, C57, C59: 1uF 250V, symbol Device:C
- removed C52, C53: 4.7uF, symbol Device:C
- removed C61: 8.2nF, symbol Device:C
- removed D17, D18, D19, D20: RSX501LAM20TR, RSX501LAM20TR:DIOM4725X105N, symbol RSX501LAM20TR:RSX501LAM20TR
- removed L10, L11, L9: 150uH, symbol Device:L
- removed L12, L13, L4, L5, L6, L7, L8: 68uH, symbol Device:L
- removed Q1, Q2: FDMC86240, FDMC86139P, symbol FDMC86240:FDMC86240
- removed R47: 3.3k, symbol Device:R_US
- removed R48, R52: 150k, symbol Device:R_US
- removed R49, R54: 10mOhm, symbol Device:R_US
- removed R50: 100K, symbol Device:R_US
- removed R51, R56: 1K, symbol Device:R_US
- removed R53: 570R, symbol Device:R_US
- removed R55: 49.9K, symbol Device:R_US
- removed U1, U2: LM5155DSSR, LM5155DSSR:IC_LM5155DSSR, symbol LM5155DSSR:LM5155DSSR
- added C100, C101, C102, C103, C104, C106, C107, C64, C65, C93, C99: 1uF, symbol Device:C
- added C30, C84, C85: 4.7uF, symbol Device:C
- added C87, C94: 100nF, symbol Device:C
- added C95, C96, C98: 47uF, symbol Device:C
- added C97: 22pF, symbol Device:C
- added FB1, FB2, FB3, FB4, FB5, FB6, FB7, FB8: BLM15AG601SN1D, symbol Device:FerriteBead
- added JP1: CLK_PWR_JMP, TMLF-6_MT_MCH, symbol Jumper:SolderJumper_2_Open
- added L17: 1uH, symbol Device:L
- added R16: 4K, symbol Device:R_US
- added R17: 1K, symbol Device:R_US
- added R34: 100K, symbol Device:R_US
- added R37: 147K, symbol Device:R_US
- added R38: 20K, symbol Device:R_US
- added R62: 10K, symbol Device:R_US
- added U15: TPS51385RJNR, VQFN-HR12_RJN_TEX, symbol TPS51385RJNR:TPS51385RJNR
- added U16, U18, U20, U22: NCP176BMX180TCG, NCP176BMX180TCG:PSON40P120X120X45-7N_NCP176BMX180TCG, symbol NCP176BMX180TCG:NCP176BMX180TCG
- added U17, U19, U21, U23: NCP176AMX330TCG, NCP176AMX330TCG:PSON40P120X120X45-7N_NCP176AMX330TCG, symbol NCP176AMX330TCG:NCP176AMX330TCG
- added U3: MIC5363-3.3YMT-TR, TMLF-6_MT_MCH, symbol MIC5363-3-3YMT-TR:MIC5363-3.3YMT-TR
Connections:
- net DC_MAIN: now also C30.1, C84.1, C85.1, C87.1, R16.1, U15.1 (VIN)
- net GND: now also C100.2, C101.2, C102.2, C103.2, C104.2, C106.2, C107.2, C30.2, C64.2, C65.2, C84.2, C85.2, C87.2, C93.2, C95.2, C96.2, C98.2, C99.2, R17.2, R38.2, R62.2, U15.10 (AGND), U15.12 (MODE), U15.2 (PGND), U16.3 (GND), U16.7 (EXP), U17.3 (GND), U17.7 (EXP), U18.3 (GND), U18.7 (EXP), U19.3 (GND), U19.7 (EXP), U20.3 (GND), U20.7 (EXP), U21.3 (GND), U21.7 (EXP), U22.3 (GND), U22.7 (EXP), U23.3 (GND), U23.7 (EXP), U3.3 (GND), U3.7 (EP)
- new net AFE1_1V8A: FB1.2
- new net AFE1_1V8D: FB1.1, U16.1 (OUT), U16.2 (FB)
- new net AFE1_1V8_EN: U16.4 (EN)
- new net AFE1_3V3A: FB2.2
- new net AFE1_3V3D: FB2.1, U17.1 (OUT), U17.2 (FB)
- new net AFE1_3V3_EN: U17.4 (EN)
- new net AFE2_1V8A: FB3.2
- new net AFE2_1V8D: FB3.1, U18.1 (OUT), U18.2 (FB)
- new net AFE2_1V8_EN: U18.4 (EN)
- new net AFE2_3V3A: FB4.2
- new net AFE2_3V3D: FB4.1, U19.1 (OUT), U19.2 (FB)
- new net AFE2_3V3_EN: U19.4 (EN)
- new net AFE3_1V8A: FB5.2
- new net AFE3_1V8D: FB5.1, U20.1 (OUT), U20.2 (FB)
- new net AFE3_1V8_EN: U20.4 (EN)
- new net AFE3_3V3A: FB6.2
- new net AFE3_3V3D: FB6.1, U21.1 (OUT), U21.2 (FB)
- new net AFE3_3V3_EN: U21.4 (EN)
- new net AFE4_1V8A: FB7.2
- new net AFE4_1V8D: FB7.1, U22.1 (OUT), U22.2 (FB)
- new net AFE4_1V8_EN: U22.4 (EN)
- new net AFE4_3V3A: FB8.2
- new net AFE4_3V3D: FB8.1, U23.1 (OUT), U23.2 (FB)
- new net AFE4_3V3_EN: U23.4 (EN)
- new net CLK_PWR_EN: R62.1, U3.6 (EN)
- new net CLK_VCC_PRE: C64.1, JP1.1 (A), U3.5 (VOUT)
- new net FANOUT_VCC: JP1.2 (B)
- new net IM_5V: C100.1, C101.1, C102.1, C103.1, C104.1, C106.1, C107.1, C65.1, C95.1, C96.1, C97.1, C98.1, C99.1, L17.2, R37.1, U16.6 (IN), U17.6 (IN), U18.6 (IN), U19.6 (IN), U20.6 (IN), U21.6 (IN), U22.6 (IN), U23.6 (IN), U3.4 (VIN)
- new net IM_5V_BS: C94.1, U15.8 (VBST)
- new net IM_5V_EN: R16.2, R17.1, U15.11 (EN)
- new net IM_5V_FB: C97.2, R37.2, R38.1, U15.4 (FB)
- new net IM_5V_PG: R34.2, U15.3 (PG)
- new net IM_5V_SW: C94.2, L17.1, U15.7 (SW)
- new net IM_5V_VCC: C93.1, U15.9 (VCC)
- no-connect marks 1 -> 10
Other:
- sheet 3V3_BUCK renamed SOM_HDC_3V3
- added sheet 100V_SUPPLY (100V_Supply.kicad_sch)
- added sheet 50V_SUPPLY (50V_Supply.kicad_sch)
- added sheet SD_CARD_3V3 (3V3_BUCK.kicad_sch)
- added sheet SOM_HDA_3V3 (3V3_BUCK.kicad_sch)
- added sheet SOM_HPA_1V8 (1V8_BUCK.kicad_sch)
- note added: "+/-100V"
- note added: "+/-50V"
- note added: "1V8 Bucks"
- note added: "3V3 Bucks"
- note added: "= 52 + 48 + 10 + 8 = 120 mA"
- note added: "AFE 1 Supplies"
- note added: "AFE 2 Supplies"
- note added: "AFE 3 Supplies"
- note added: "AFE 4 Supplies"
- note added: "Fanout Buffer 3V3"
- note added: "HV Supplies (+/- 50/100V)"
- note added: "Intermediate 5V Supply"
- note added: "Main SOM 5V Supply"
- note added: "Miscellaneous Supplies"
- note added: "Processing Section (PL) Supplies"
- note added: "Pulser 1V8"
- note added: "USB 1V8"
- note added: "^ x4 = 1.2A"
- note removed: "= (0.3*100.7*1.2) / (11*0.88) = 3.75A"
- note removed: "= (100+0.7) / (11+100+0.7) = 90%"
- note removed: "= (11*25*0.9) / (2*0.3*100*0.4*150000) = 68uH"
- note removed: "= (50+0.7) / (11+50+0.7) = 82%"
- note removed: "= 0.3 * 1.2 = 0.36A"
- note removed: "= 146k (approx. 150k)"
- note removed: "Cs1 = Cs2 = 2.2uF"
- note removed: "Cs1 = Cs2 = 3.9uF"
- note removed: "F_switching = 150 KHz"
- note removed: "R_fbt = 99k/49 (approx. 100k/49.9) R_fbb = 1k"
- note removed: "Rcomp = 3.3k, Ccomp = 46nF R_HF = 8.2nF"
- note removed: "n = 0.88"
- moved on the sheet: C10, C44, C8, C9

Commit message: DONE! hust needs a final revision, checking termination throughout the circuit and verifying the signal chain
Parts:
- removed C10, C8, C9, C95, C96, C98: 47uF, symbol Device:C
- removed C30, C4, C5, C6: 4.7uF, symbol Device:C
- removed C43, C45, C87, C94: 100nF, symbol Device:C
- removed C44, C93: 1uF, symbol Device:C
- removed C7, C97: 22pF, symbol Device:C
- removed L1: 1uH, symbol Device:L
- removed R10, R34: 100K, symbol Device:R_US
- removed R16, R7: 4K, symbol Device:R_US
- removed R17, R6: 1K, symbol Device:R_US
- removed R37, R8: 147K, symbol Device:R_US
- removed R38, R9: 20K, symbol Device:R_US
- removed U15, U8: TPS51385RJNR, VQFN-HR12_RJN_TEX, symbol TPS51385RJNR:TPS51385RJNR
- added C229: 10uF, Capacitor_SMD:C_0805_2012Metric, symbol Device:C
- added C230: 100nF, symbol Device:C
- added C231: 220nF, symbol Device:C
- added C232: 4.7nF, Capacitor_SMD:C_0603_1608Metric, symbol Device:C
- added C233: 10pF, symbol Device:C
- added C234: 22uF, Capacitor_SMD:C_0805_2012Metric, symbol Device:C
- added D10, D11, D12, D14, D15, D2, D4, D6, D7, D8: LED, symbol Device:LED
- added D3: B240A-13-F, digikey-footprints:DO-214AC, symbol dk_Diodes-Rectifiers-Single:B240A-13-F
- added R103, R76, R81, R82, R83, R84, R85, R86, R87, R88: 10K, symbol Device:R_US
- added R77: 10R, symbol Device:R_US
- added R78: 100K, symbol Device:R_US
- added R79: 150K, symbol Device:R_US
- added R80: 619K, symbol Device:R_US
- added R89: 1K, symbol Device:R_US
- added R90, R91: 0.5K, symbol Device:R_US
- added R92, R93, R94, R95: 330R, symbol Device:R_US
- added R96, R97, R98: 220R, symbol Device:R_US
- added U15: TPS63700DRCR, TPS63700DRCR:VREG_V62_16624-01YE, symbol TPS63700DRCR:TPS63700DRCR
- added U31: NCP176BMX180TCG, NCP176BMX180TCG:PSON40P120X120X45-7N_NCP176BMX180TCG, symbol NCP176BMX180TCG:NCP176BMX180TCG
- added U6: TPS22918TDBVRQ1, TPS22918TDBVRQ1:SOT95P280X145-6N, symbol TPS22918TDBVRQ1:TPS22918TDBVRQ1
- C84, C85: value 4.7uF -> 1uF
- L17: value 1uH -> 4.7uH; footprint (none) -> Inductor_SMD:L_0805_2012Metric
Connections:
- net IM_5V_SW is gone; now on net GND: L17.1
- net AFE1_1V8_EN: now also R81.1
- net AFE1_3V3_EN: now also R82.1
- net AFE2_1V8_EN: now also R83.1
- net AFE2_3V3_EN: now also R84.1
- net AFE3_1V8_EN: now also R103.1, R85.1, U31.4 (EN)
- net AFE3_3V3_EN: now also R86.1
- net AFE4_1V8_EN: now also R87.1
- net AFE4_3V3_EN: now also R88.1
- net CLK_VCC_PRE: now also R95.1
- net DC_MAIN: now also R89.1; no longer C84.1, C85.1
- net GND: now also C229.2, C230.2, C231.2, C232.2, C234.2, D10.1 (K), D11.1 (K), D12.1 (K), D14.1 (K), D15.1 (K), D2.1 (K), D4.1 (K), D6.1 (K), D7.1 (K), D8.1 (K), R103.2, R76.2, R81.2, R82.2, R83.2, R84.2, R85.2, R86.2, R87.2, R88.2, U15.11 (EP), U15.2 (GND), U15.7 (PS_GND), U31.3 (GND), U31.7 (EXP), U6.2 (GND)
- net IM_5V: now also C229.1, R77.1, R90.1, U15.5 (IN), U31.6 (IN); no longer L17.2
- net PULSER_1V8: now also C85.1, R97.1, U6.5 (QOD), U6.6 (VOUT)
- net PULSER_1V8_EN: now also U6.3 (ON)
- net SD_3V3: now also R92.1
- net SOM_5V: now also R91.1
- net USB_1V8: now also C84.1, R96.1, U6.1 (VIN)
- net VDD_HDA: now also R93.1
- net VDD_HDB: now also R94.1
- net VDD_HPA: now also R98.1
- new net: D12.2 (A), R91.2
- new net: C233.2, R78.1
- new net: D4.2 (A), R97.2
- new net: D7.2 (A), R95.2
- new net: D2.2 (A), R98.2
- new net: D11.2 (A), R92.2
- new net: D14.2 (A), R90.2
- new net: D10.2 (A), R93.2
- new net: D8.2 (A), R94.2
- new net: D6.2 (A), R96.2
- new net: D15.2 (A), R89.2
- new net: C230.1, R77.2, U15.3 (VIN)
- new net -5V_EN: R76.1, U15.4 (EN)
- new net -5_COMP: C232.1, U15.1 (COMP)
- new net -5_FB: C233.1, R79.1, R80.2, U15.9 (FB)
- new net -5_SW: D3.K, L17.2, U15.6 (SW)
- new net -5_VREF: C231.1, R79.2, U15.10 (VREF)
- new net CLK_1V8: U31.1 (OUT), U31.2 (FB)
- new net PULSER_5VN: C234.1, D3.A, R78.2, R80.1, U15.8 (OUT)
- no-connect marks 10 -> 11
Other:
- removed sheet TX1V8
- added sheet IM_5V (5V_BUCK.kicad_sch)
- added sheet SOM_5V (5V_BUCK.kicad_sch)
- note added: "Pulser + Intermediate 5V Supply"
- note added: "Pulser + USB 1V8"
- note added: "Pulser -5V Supply"
- note added: "SD Card 3V3"
- note added: "The LC-filter at Vin is recommended by the datasheet."
- note added: "The values of the: - Compensation capacitor (4.7nF) - Inductor (4.7uH for -5V) - Output capacitor (>12uF) - Voltage divider - Feed-forward network Were recommended by the datasheet"
- note removed: "- Change values as long as they're 1:4 - Maintain low tolerance & low heat-coefficient - 0.2 * 12 = 2.4 (HIGH) - 0.2 * 24 = 4.8 (HIGH)"
- note removed: "Intermediate 5V Supply"
- note removed: "Pulser 1V8"
- note removed: "USB 1V8"
- note removed: "WeBench Designer Link"
- moved on the sheet: C64, C65, JP1, R62, U3

Commit message: HDMI was requested so add it and give the signal chain a final revision
Parts:
- added C182, C218, C239: 1uF, symbol Device:C
- added U26: NCP176AMX330TCG, NCP176AMX330TCG:PSON40P120X120X45-7N_NCP176AMX330TCG, symbol NCP176AMX330TCG:NCP176AMX330TCG
Connections:
- net AFE2_1V8_EN is gone; now on net AFE_1V8_EN: R83.1, U18.4 (EN)
- net AFE2_3V3_EN is gone; now on net AFE_3V3_EN: R84.1, U19.4 (EN)
- net AFE3_3V3_EN is gone; now on net AFE_3V3_EN: R86.1, U21.4 (EN)
- net AFE4_1V8_EN is gone; now on net AFE_1V8_EN: R87.1, U22.4 (EN)
- net AFE4_3V3_EN is gone; now on net AFE_3V3_EN: R88.1, U23.4 (EN)
- net GND: now also C182.2, C218.2, C239.2, U26.3 (GND), U26.7 (EXP)
- net IM_5V: now also C218.1, C239.1, U26.4 (EN), U26.6 (IN)
- net AFE1_1V8_EN renamed AFE_1V8_EN
- net AFE_1V8_EN: now also R85.1, U20.4 (EN)
- net AFE1_3V3_EN renamed AFE_3V3_EN
- net AFE3_1V8_EN renamed CLK_1V8_EN
- net CLK_1V8_EN: no longer R85.1, U20.4 (EN)
- new net EXT_3V3: C182.1, U26.1 (OUT), U26.2 (FB)
- no-connect marks 11 -> 12
Other:
- moved on the sheet: R103, U31

Commit message: ALL IS DONE EXCEPT HDMI PLEASE HELP
Parts:
- removed R83, R84, R85, R86, R87, R88: 10K, symbol Device:R_US
- removed U18, U22: NCP176BMX180TCG, NCP176BMX180TCG:PSON40P120X120X45-7N_NCP176BMX180TCG, symbol NCP176BMX180TCG:NCP176BMX180TCG
- removed U19, U23: NCP176AMX330TCG, NCP176AMX330TCG:PSON40P120X120X45-7N_NCP176AMX330TCG, symbol NCP176AMX330TCG:NCP176AMX330TCG
- added C244, C245: 1uF, symbol Device:C
- added JP10, JP11: SD_3V3_JMP, TMLF-6_MT_MCH, symbol Jumper:SolderJumper_2_Open
- added JP12: -5V_JMP, TMLF-6_MT_MCH, symbol Jumper:SolderJumper_2_Open
- added JP13: SOM_5V_JMP, TMLF-6_MT_MCH, symbol Jumper:SolderJumper_2_Open
- added JP6: IM_5V_JMP, TMLF-6_MT_MCH, symbol Jumper:SolderJumper_2_Open
- added JP7: HDA_3V3_JMP, TMLF-6_MT_MCH, symbol Jumper:SolderJumper_2_Open
- added JP8: HDBC_3V3_JMP, TMLF-6_MT_MCH, symbol Jumper:SolderJumper_2_Open
- added JP9: HPA_1V8_JMP, TMLF-6_MT_MCH, symbol Jumper:SolderJumper_2_Open
- added R66: 10K, symbol Device:R_US
- added U30: NCP176AMX330TCG, NCP176AMX330TCG:PSON40P120X120X45-7N_NCP176AMX330TCG, symbol NCP176AMX330TCG:NCP176AMX330TCG
Connections:
- net AFE2_1V8D is gone; now on net AFE1_1V8D: FB3.1
- net AFE2_3V3D is gone; now on net AFE1_3V3D: FB4.1
- net AFE4_1V8D is gone; now on net AFE3_1V8D: FB7.1
- net AFE4_3V3D is gone; now on net AFE3_3V3D: FB8.1
- net GND: now also C244.2, C245.2, R66.2, U30.3 (GND), U30.7 (EXP)
- net PULSER_1V8_EN: now also R66.1
- net PULSER_5VN: now also JP12.2 (B); no longer C234.1, D3.A, R78.2, R80.1, U15.8 (OUT)
- net SD_3V3: now also JP10.2 (B)
- net SOM_5V: now also JP13.2 (B)
- net USB_1V8: now also JP11.2 (B)
- net VDD_HDA: now also JP7.2 (B)
- net VDD_HDB: now also JP8.2 (B)
- net VDD_HPA: now also JP9.2 (B)
- net FANOUT_VCC renamed CLK_3V3
- net IM_5V renamed HDMI_5V
- net HDMI_5V: now also C244.1, JP6.2 (B), U30.4 (EN), U30.6 (IN)
- new net HDMI_3V3: C245.1, U30.1 (OUT), U30.2 (FB)
- new net IM_5V_PRE: JP6.1 (A)
- new net PULSER_5VN_PRE: C234.1, D3.A, JP12.1 (A), R78.2, R80.1, U15.8 (OUT)
- new net SD_3V3_PRE: JP10.1 (A)
- new net SOM_5V_PRE: JP13.1 (A)
- new net USB_1V8_PRE: JP11.1 (A)
- new net VDD_HDA_PRE: JP7.1 (A)
- new net VDD_HDBC_PRE: JP8.1 (A)
- new net VDD_HPA_PRE: JP9.1 (A)
- no-connect marks 12 -> 9
Other:
- note added: "AFE 1 & 2 Supplies"
- note added: "AFE 3 & 4 Supplies"
- note added: "AFE LDOs (1.8V & 3V3)"
- note added: "CLOCK 1V8"
- note added: "CLOCK 3V3"
- note added: "External Interfaces 3V3"
- note added: "HDMI 3V3"
- note removed: "AFE 1 Supplies"
- note removed: "AFE 2 Supplies"
- note removed: "AFE 3 Supplies"
- note removed: "AFE 4 Supplies"
- note removed: "Fanout Buffer 3V3"
- moved on the sheet: C100, C101, C102, C103, C104, C106, C107, C182, C218, C229, C230, C231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
