File: Power.kicad_sch (KiCad schematic)
At the start: 82 parts, among them U15 TPS63700DRCR, U16 NCP176BMX180TCG, U17 NCP176AMX330TCG, U20 NCP176BMX180TCG, U21 NCP176AMX330TCG, U26 NCP176AMX330TCG, U3 MIC5363-3.3YMT-TR, U30 NCP176AMX330TCG, U31 NCP176BMX180TCG, U6 TPS22918TDBVRQ1

Commit message: started layout, finished 90% of individual section placement, need to finish remaining and integrate together in PCB and apply schematic edits before
Parts:
- removed C103, C104, C106, C107, C244, C245: 1uF, symbol Device:C
- removed U30: NCP176AMX330TCG, NCP176AMX330TCG:PSON40P120X120X45-7N_NCP176AMX330TCG, symbol NCP176AMX330TCG:NCP176AMX330TCG
- added C411: 1uF, Capacitor_SMD:C_0402_1005Metric, symbol Device:C
- added R421: 10K, Resistor_SMD:R_0402_1005Metric, symbol Device:R_US
- C402: renamed from C230; footprint (none) -> Capacitor_SMD:C_0402_1005Metric
- C403: renamed from C231; footprint (none) -> Capacitor_SMD:C_0402_1005Metric
- C405: renamed from C233; footprint (none) -> Capacitor_SMD:C_0402_1005Metric
- C407: renamed from C99; footprint (none) -> Capacitor_SMD:C_0402_1005Metric
- C408: renamed from C100; footprint (none) -> Capacitor_SMD:C_0402_1005Metric
- C409: renamed from C101; footprint (none) -> Capacitor_SMD:C_0402_1005Metric
- C410: renamed from C102; footprint (none) -> Capacitor_SMD:C_0402_1005Metric
- C415: renamed from C239; footprint (none) -> Capacitor_SMD:C_0402_1005Metric
- C416: renamed from C65; footprint (none) -> Capacitor_SMD:C_0402_1005Metric
- C417: renamed from C218; footprint (none) -> Capacitor_SMD:C_0402_1005Metric
- C419: renamed from C84; footprint (none) -> Capacitor_SMD:C_0402_1005Metric
- C420: renamed from C64; footprint (none) -> Capacitor_SMD:C_0402_1005Metric
- C421: renamed from C85; footprint (none) -> Capacitor_SMD:C_0402_1005Metric
- C422: renamed from C182; footprint (none) -> Capacitor_SMD:C_0402_1005Metric
- D401: renamed from D15; footprint (none) -> LED_SMD:LED_0603_1608Metric
- D402: renamed from D14; footprint (none) -> LED_SMD:LED_0603_1608Metric
- D403: renamed from D12; footprint (none) -> LED_SMD:LED_0603_1608Metric
- D404: renamed from D11; footprint (none) -> LED_SMD:LED_0603_1608Metric
- D405: renamed from D10; footprint (none) -> LED_SMD:LED_0603_1608Metric
- D406: renamed from D8; footprint (none) -> LED_SMD:LED_0603_1608Metric
- D407: renamed from D7; footprint (none) -> LED_SMD:LED_0603_1608Metric
- D409: renamed from D6; footprint (none) -> LED_SMD:LED_0603_1608Metric
- D410: renamed from D4; footprint (none) -> LED_SMD:LED_0603_1608Metric
- D411: renamed from D2; footprint (none) -> LED_SMD:LED_0603_1608Metric
- FB401: renamed from FB1; footprint (none) -> Inductor_SMD:L_0402_1005Metric
- FB402: renamed from FB2; footprint (none) -> Inductor_SMD:L_0402_1005Metric
- FB403: renamed from FB7; footprint (none) -> Inductor_SMD:L_0402_1005Metric
- FB404: renamed from FB3; footprint (none) -> Inductor_SMD:L_0402_1005Metric
- FB405: renamed from FB4; footprint (none) -> Inductor_SMD:L_0402_1005Metric
- FB406: renamed from FB8; footprint (none) -> Inductor_SMD:L_0402_1005Metric
- FB407: renamed from FB5; footprint (none) -> Inductor_SMD:L_0402_1005Metric
- FB408: renamed from FB6; footprint (none) -> Inductor_SMD:L_0402_1005Metric
- JP401: renamed from JP6; footprint TMLF-6_MT_MCH -> Jumper:SolderJumper-2_P1.3mm_Open_TrianglePad1.0x1.5mm
- JP402: renamed from JP13; footprint TMLF-6_MT_MCH -> Jumper:SolderJumper-2_P1.3mm_Open_TrianglePad1.0x1.5mm
- JP403: renamed from JP12; footprint TMLF-6_MT_MCH -> Jumper:SolderJumper-2_P1.3mm_Open_TrianglePad1.0x1.5mm
- JP404: renamed from JP8; footprint TMLF-6_MT_MCH -> Jumper:SolderJumper-2_P1.3mm_Open_TrianglePad1.0x1.5mm
- JP405: renamed from JP7; footprint TMLF-6_MT_MCH -> Jumper:SolderJumper-2_P1.3mm_Open_TrianglePad1.0x1.5mm
- JP406: renamed from JP9; footprint TMLF-6_MT_MCH -> Jumper:SolderJumper-2_P1.3mm_Open_TrianglePad1.0x1.5mm
- JP407: renamed from JP11; footprint TMLF-6_MT_MCH -> Jumper:SolderJumper-2_P1.3mm_Open_TrianglePad1.0x1.5mm
- JP408: renamed from JP10; footprint TMLF-6_MT_MCH -> Jumper:SolderJumper-2_P1.3mm_Open_TrianglePad1.0x1.5mm
- JP409: renamed from JP1; footprint TMLF-6_MT_MCH -> Jumper:SolderJumper-2_P1.3mm_Open_TrianglePad1.0x1.5mm
- R401: renamed from R89; footprint (none) -> Resistor_SMD:R_0402_1005Metric
- R402: renamed from R76; footprint (none) -> Resistor_SMD:R_0402_1005Metric
- R403: renamed from R90; footprint (none) -> Resistor_SMD:R_0402_1005Metric
- R404: renamed from R77; footprint (none) -> Resistor_SMD:R_0402_1005Metric
- R405: renamed from R91; footprint (none) -> Resistor_SMD:R_0402_1005Metric
- R406: renamed from R92; footprint (none) -> Resistor_SMD:R_0402_1005Metric
- R407: renamed from R93; footprint (none) -> Resistor_SMD:R_0402_1005Metric
- R408: renamed from R94; footprint (none) -> Resistor_SMD:R_0402_1005Metric
- R409: renamed from R95; footprint (none) -> Resistor_SMD:R_0402_1005Metric
- R410: renamed from R79; footprint (none) -> Resistor_SMD:R_0402_1005Metric
- R411: renamed from R80; footprint (none) -> Resistor_SMD:R_0402_1005Metric
- R412: renamed from R96; footprint (none) -> Resistor_SMD:R_0402_1005Metric
- R413: renamed from R78; footprint (none) -> Resistor_SMD:R_0402_1005Metric
- R414: renamed from R97; footprint (none) -> Resistor_SMD:R_0402_1005Metric
- R415: renamed from R98; footprint (none) -> Resistor_SMD:R_0402_1005Metric
- R416: renamed from R81; footprint (none) -> Resistor_SMD:R_0402_1005Metric
- R417: renamed from R82; footprint (none) -> Resistor_SMD:R_0402_1005Metric
- R418: renamed from R103; footprint (none) -> Resistor_SMD:R_0402_1005Metric
- R419: renamed from R62; footprint (none) -> Resistor_SMD:R_0402_1005Metric
- R420: renamed from R66; footprint (none) -> Resistor_SMD:R_0402_1005Metric
- U407: renamed from U3; footprint TMLF-6_MT_MCH -> MIC5363-3-3YMT-TR:TMLF-6_MT_MCH
- renumbered C229 to C401, C232 to C404, C234 to C406, D3 to D408, L17 to L401, U15 to U401, U16 to U402, U17 to U403, U20 to U404, U21 to U405, U31 to U406, U26 to U408, U6 to U410
Connections:
- net CLK_1V8: now also C411.1
- net GND: now also C411.2, R421.2
- net SOM_PL_PWR_EN: now also R421.1
- net HDMI_5V renamed IM_5V
- no-connect marks 9 -> 8
Other:
- note removed: "HDMI 3V3"
