File: 1V8_BUCK.kicad_sch (KiCad schematic)
At the start: 10 parts, among them U6 TPS54302

Commit message: DONE! hust needs a final revision, checking termination throughout the circuit and verifying the signal chain
Parts:
- renumbered C47 to C222, C50 to C223, C48 to C224, C49 to C225, C13 to C27, C16 to C28, L3 to L14, R44 to R46, R45 to R60, U6 to U14
Changed lines of the file:
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@@
 		(dnp no)
 		(fields_autoplaced yes)
-		(property "Reference" "U6"
+		(property "Reference" "U14"
 			(at 121.92 83.82 0)
 			(show_name no)
@@
 		(instances
 			(project "MedicalImager"
-				(path "/99848109-7be9-4113-bc9c-faf6c2acfe0b/bd63d6e1-5dfb-4921-86f2-9a66ea07210d/1acf250f-5047-45dc-9a16-165524a78292"
-					(reference "U6")
-					(unit 1)
-				)
 				(path "/99848109-7be9-4113-bc9c-faf6c2acfe0b/bd63d6e1-5dfb-4921-86f2-9a66ea07210d/6035e4a1-a138-4208-abfe-cd2d572bc56c"
 					(reference "U12")
@@
 		(dnp no)
 		(fields_autoplaced yes)
-		(property "Reference" "#PWR0178"
+		(property "Reference" "#PWR0222"
 			(at 121.92 110.49 0)
 			(hide yes)
@@
 		(instances
 			(project "MedicalImager"
-				(path "/99848109-7be9-4113-bc9c-faf6c2acfe0b/bd63d6e1-5dfb-4921-86f2-9a66ea07210d/1acf250f-5047-45dc-9a16-165524a78292"
-					(reference "#PWR0178")
-					(unit 1)
-				)
 				(path "/99848109-7be9-4113-bc9c-faf6c2acfe0b/bd63d6e1-5dfb-4921-86f2-9a66ea07210d/6035e4a1-a138-4208-abfe-cd2d572bc56c"
 					(reference "#PWR0241")
@@
 		(dnp no)
 		(fields_autoplaced yes)
-		(property "Reference" "R44"
+		(property "Reference" "R46"
 			(at 161.29 100.3299 0)
 			(show_name no)
@@
 		(instances
 			(project "MedicalImager"
-				(path "/99848109-7be9-4113-bc9c-faf6c2acfe0b/bd63d6e1-5dfb-4921-86f2-9a66ea07210d/1acf250f-5047-45dc-9a16-165524a78292"
-					(reference "R44")
-					(unit 1)
-				)
 				(path "/99848109-7be9-4113-bc9c-faf6c2acfe0b/bd63d6e1-5dfb-4921-86f2-9a66ea07210d/6035e4a1-a138-4208-abfe-cd2d572bc56c"
 					(reference "R63")
@@
 		(dnp no)
 		(fields_autoplaced yes)
-		(property "Reference" "#PWR0182"
+		(property "Reference" "#PWR0224"
 			(at 196.85 123.19 0)
 			(hide yes)
@@
 		(instances
 			(project "MedicalImager"
-				(path "/99848109-7be9-4113-bc9c-faf6c2acfe0b/bd63d6e1-5dfb-4921-86f2-9a66ea07210d/1acf250f-5047-45dc-9a16-165524a78292"
-					(reference "#PWR0182")
-					(unit 1)
-				)
 				(path "/99848109-7be9-4113-bc9c-faf6c2acfe0b/bd63d6e1-5dfb-4921-86f2-9a66ea07210d/6035e4a1-a138-4208-abfe-cd2d572bc56c"
 					(reference "#PWR0243")
@@
 		(dnp no)
 		(fields_autoplaced yes)
-		(property "Reference" "C49"
+		(property "Reference" "C225"
 			(at 207.01 106.6799 0)
 			(show_name no)
@@
 		(instances
 			(project "MedicalImager"
-				(path "/99848109-7be9-4113-bc9c-faf6c2acfe0b/bd63d6e1-5dfb-4921-86f2-9a66ea07210d/1acf250f-5047-45dc-9a16-165524a78292"
-					(reference "C49")
-					(unit 1)
-				)
 				(path "/99848109-7be9-4113-bc9c-faf6c2acfe0b/bd63d6e1-5dfb-4921-86f2-9a66ea07210d/6035e4a1-a138-4208-abfe-cd2d572bc56c"
 					(reference "C83")
@@
 		(dnp no)
 		(fields_autoplaced yes)
-		(property "Reference" "C50"
+		(property "Reference" "C223"
 			(at 175.26 100.3299 0)
 			(show_name no)
@@
 		(instances
 			(project "MedicalImager"
-				(path "/99848109-7be9-4113-bc9c-faf6c2acfe0b/bd63d6e1-5dfb-4921-86f2-9a66ea07210d/1acf250f-5047-45dc-9a16-165524a78292"
-					(reference "C50")
-					(unit 1)
-				)
 				(path "/99848109-7be9-4113-bc9c-faf6c2acfe0b/bd63d6e1-5dfb-4921-86f2-9a66ea07210d/6035e4a1-a138-4208-abfe-cd2d572bc56c"
 					(reference "C76")
@@
 		(dnp no)
 		(fields_autoplaced yes)
-		(property "Reference" "R45"
+		(property "Reference" "R60"
 			(at 161.29 113.0299 0)
 			(show_name no)
@@
 		(instances
 			(project "MedicalImager"
-				(path "/99848109-7be9-4113-bc9c-faf6c2acfe0b/bd63d6e1-5dfb-4921-86f2-9a66ea07210d/1acf250f-5047-45dc-9a16-165524a78292"
-					(reference "R45")
-					(unit 1)
-				)
 				(path "/99848109-7be9-4113-bc9c-faf6c2acfe0b/bd63d6e1-5dfb-4921-86f2-9a66ea07210d/6035e4a1-a138-4208-abfe-cd2d572bc56c"
 					(reference "R64")
@@
 		(dnp no)
 		(fields_autoplaced yes)
-		(property "Reference" "C48"
+		(property "Reference" "C224"
 			(at 194.31 106.6799 0)
 			(show_name no)
@@
 		(instances
 			(project "MedicalImager"
-				(path "/99848109-7be9-4113-bc9c-faf6c2acfe0b/bd63d6e1-5dfb-4921-86f2-9a66ea07210d/1acf250f-5047-45dc-9a16-165524a78292"
-					(reference "C48")
-					(unit 1)
-				)
 				(path "/99848109-7be9-4113-bc9c-faf6c2acfe0b/bd63d6e1-5dfb-4921-86f2-9a66ea07210d/6035e4a1-a138-4208-abfe-cd2d572bc56c"
 					(reference "C77")
@@
 		(in_pos_files yes)
 		(dnp no)
-		(property "Reference" "C47"
+		(property "Reference" "C222"
 			(at 135.89 81.2799 0)
 			(show_name no)
@@
 		(instances
 			(project "MedicalImager"
-				(path "/99848109-7be9-4113-bc9c-faf6c2acfe0b/bd63d6e1-5dfb-4921-86f2-9a66ea07210d/1acf250f-5047-45dc-9a16-165524a78292"
-					(reference "C47")
-					(unit 1)
-				)
 				(path "/99848109-7be9-4113-bc9c-faf6c2acfe0b/bd63d6e1-5dfb-4921-86f2-9a66ea07210d/6035e4a1-a138-4208-abfe-cd2d572bc56c"
 					(reference "C72")
@@
 		(dnp no)
 		(fields_autoplaced yes)
-		(property "Reference" "#PWR0180"
+		(property "Reference" "#PWR0223"
 			(at 158.75 127 0)
 			(hide yes)
@@
 		(instances
 			(project "MedicalImager"
-				(path "/99848109-7be9-4113-bc9c-faf6c2acfe0b/bd63d6e1-5dfb-4921-86f2-9a66ea07210d/1acf250f-5047-45dc-9a16-165524a78292"
-					(reference "#PWR0180")
-					(unit 1)
-				)
 				(path "/99848109-7be9-4113-bc9c-faf6c2acfe0b/bd63d6e1-5dfb-4921-86f2-9a66ea07210d/6035e4a1-a138-4208-abfe-cd2d572bc56c"
 					(reference "#PWR0242")
@@
 		(dnp no)
 		(fields_autoplaced yes)
-		(property "Reference" "#PWR0176"
+		(property "Reference" "#PWR0221"
 			(at 95.25 123.19 0)
 			(hide yes)
@@
 		(instances
 			(project "MedicalImager"
-				(path "/99848109-7be9-4113-bc9c-faf6c2acfe0b/bd63d6e1-5dfb-4921-86f2-9a66ea07210d/1acf250f-5047-45dc-9a16-165524a78292"
-					(reference "#PWR0176")
-					(unit 1)
-				)
 				(path "/99848109-7be9-4113-bc9c-faf6c2acfe0b/bd63d6e1-5dfb-4921-86f2-9a66ea07210d/6035e4a1-a138-4208-abfe-cd2d572bc56c"
 					(reference "#PWR0214")
@@
 		(dnp no)
 		(fields_autoplaced yes)
-		(property "Reference" "C13"
+		(property "Reference" "C27"
 			(at 92.71 106.6799 0)
 			(show_name no)
@@
 		(instances
 			(project "MedicalImager"
-				(path "/99848109-7be9-4113-bc9c-faf6c2acfe0b/bd63d6e1-5dfb-4921-86f2-9a66ea07210d/1acf250f-5047-45dc-9a16-165524a78292"
-					(reference "C13")
-					(unit 1)
-				)
 				(path "/99848109-7be9-4113-bc9c-faf6c2acfe0b/bd63d6e1-5dfb-4921-86f2-9a66ea07210d/6035e4a1-a138-4208-abfe-cd2d572bc56c"
 					(reference "C18")
@@
 		(dnp no)
 		(fields_autoplaced yes)
-		(property "Reference" "C16"
+		(property "Reference" "C28"
 			(at 105.41 106.6799 0)
 			(show_name no)
@@
 		(instances
 			(project "MedicalImager"
-				(path "/99848109-7be9-4113-bc9c-faf6c2acfe0b/bd63d6e1-5dfb-4921-86f2-9a66ea07210d/1acf250f-5047-45dc-9a16-165524a78292"
-					(reference "C16")
-					(unit 1)
-				)
 				(path "/99848109-7be9-4113-bc9c-faf6c2acfe0b/bd63d6e1-5dfb-4921-86f2-9a66ea07210d/6035e4a1-a138-4208-abfe-cd2d572bc56c"
 					(reference "C29")
@@
 		(dnp no)
 		(fields_autoplaced yes)
-		(property "Reference" "L3"
+		(property "Reference" "L14"
 			(at 152.4 88.9 90)
 			(show_name no)
@@
 		(instances
 			(project "MedicalImager"
-				(path "/99848109-7be9-4113-bc9c-faf6c2acfe0b/bd63d6e1-5dfb-4921-86f2-9a66ea07210d/1acf250f-5047-45dc-9a16-165524a78292"
-					(reference "L3")
-					(unit 1)
-				)
 				(path "/99848109-7be9-4113-bc9c-faf6c2acfe0b/bd63d6e1-5dfb-4921-86f2-9a66ea07210d/6035e4a1-a138-4208-abfe-cd2d572bc56c"
 					(reference "L15")

Commit message: started layout, finished 90% of individual section placement, need to finish remaining and integrate together in PCB and apply schematic edits before
Parts:
- C1301: renamed from C27; footprint (none) -> Capacitor_SMD:C_0805_2012Metric
- C1302: renamed from C28; footprint (none) -> Capacitor_SMD:C_0805_2012Metric
- C1303: renamed from C222; footprint (none) -> Capacitor_SMD:C_0402_1005Metric
- C1304: renamed from C223; footprint (none) -> Capacitor_SMD:C_0402_1005Metric
- C1305: renamed from C224; footprint (none) -> Capacitor_SMD:C_0805_2012Metric
- C1306: renamed from C225; footprint (none) -> Capacitor_SMD:C_0805_2012Metric
- L1301: renamed from L14; footprint (none) -> Inductor_SMD:L_6.3x6.3_H3
- R1301: renamed from R46; footprint (none) -> Resistor_SMD:R_0402_1005Metric
- R1302: renamed from R60; footprint (none) -> Resistor_SMD:R_0402_1005Metric
- renumbered U14 to U1301
