File: 3V3_BUCK.kicad_sch (KiCad schematic)
At the start: 9 parts, among them U5 TPS54302

Commit message: started layout, finished 90% of individual section placement, need to finish remaining and integrate together in PCB and apply schematic edits before
Parts:
- C1101: renamed from C11; footprint (none) -> Capacitor_SMD:C_0805_2012Metric
- C1102: renamed from C12; footprint (none) -> Capacitor_SMD:C_0805_2012Metric
- C1103: renamed from C46; footprint (none) -> Capacitor_SMD:C_0402_1005Metric
- C1104: renamed from C51; footprint (none) -> Capacitor_SMD:C_0402_1005Metric
- C1105: renamed from C15; footprint (none) -> Capacitor_SMD:C_0805_2012Metric
- L1101: renamed from L2; footprint (none) -> Inductor_SMD:L_6.3x6.3_H3
- R1101: renamed from R12; footprint (none) -> Resistor_SMD:R_0402_1005Metric
- R1102: renamed from R13; footprint (none) -> Resistor_SMD:R_0402_1005Metric
- renumbered U5 to U1101
