File: 5V_BUCK.kicad_sch (KiCad schematic)
At the start: 17 parts, among them U8 TPS51385RJNR

Commit message: started layout, finished 90% of individual section placement, need to finish remaining and integrate together in PCB and apply schematic edits before
Parts:
- C1901: renamed from C4; footprint (none) -> Capacitor_SMD:C_0805_2012Metric
- C1902: renamed from C5; footprint (none) -> Capacitor_SMD:C_0805_2012Metric
- C1903: renamed from C6; footprint (none) -> Capacitor_SMD:C_0805_2012Metric
- C1904: renamed from C7; footprint (none) -> Capacitor_SMD:C_0402_1005Metric
- C1905: renamed from C8; footprint (none) -> Capacitor_SMD:C_0402_1005Metric
- C1906: renamed from C9; footprint (none) -> Capacitor_SMD:C_0402_1005Metric
- C1907: renamed from C10; footprint (none) -> Capacitor_SMD:C_0805_2012Metric
- C1908: renamed from C43; footprint (none) -> Capacitor_SMD:C_0805_2012Metric
- C1909: renamed from C44; footprint (none) -> Capacitor_SMD:C_0402_1005Metric
- C1910: renamed from C45; footprint (none) -> Capacitor_SMD:C_0805_2012Metric
- L1901: renamed from L1; footprint (none) -> Inductor_SMD:L_10.4x10.4_H4.8
- R1901: renamed from R6; footprint (none) -> Resistor_SMD:R_0402_1005Metric
- R1902: renamed from R7; footprint (none) -> Resistor_SMD:R_0402_1005Metric
- R1903: renamed from R8; footprint (none) -> Resistor_SMD:R_0402_1005Metric
- R1904: renamed from R9; footprint (none) -> Resistor_SMD:R_0402_1005Metric
- R1905: renamed from R10; footprint (none) -> Resistor_SMD:R_0402_1005Metric
- U1901: renamed from U8; footprint VQFN-HR12_RJN_TEX -> TPS51385RJNR:VQFN-HR12_RJN_TEX
