File: RX_LANE.kicad_sch (KiCad schematic)
At the start: 42 parts, among them U7 AD8285WBCPZ

Commit message: started layout, finished 90% of individual section placement, need to finish remaining and integrate together in PCB and apply schematic edits before
Parts:
- C601: renamed from C145; footprint (none) -> Capacitor_SMD:C_0402_1005Metric
- C602: renamed from C146; footprint (none) -> Capacitor_SMD:C_0402_1005Metric
- C603: renamed from C125; footprint (none) -> Capacitor_SMD:C_0402_1005Metric
- C604: renamed from C157; footprint (none) -> Capacitor_SMD:C_0402_1005Metric
- C605: renamed from C129; footprint (none) -> Capacitor_SMD:C_0402_1005Metric
- C606: renamed from C109; footprint (none) -> Capacitor_SMD:C_0402_1005Metric
- C607: renamed from C113; footprint (none) -> Capacitor_SMD:C_0402_1005Metric
- C608: renamed from C158; footprint (none) -> Capacitor_SMD:C_0402_1005Metric
- C609: renamed from C130; footprint (none) -> Capacitor_SMD:C_0402_1005Metric
- C610: renamed from C105; footprint (none) -> Capacitor_SMD:C_0402_1005Metric
- C611: renamed from C114; footprint (none) -> Capacitor_SMD:C_0402_1005Metric
- C612: renamed from C159; footprint (none) -> Capacitor_SMD:C_0402_1005Metric
- C613: renamed from C131; footprint (none) -> Capacitor_SMD:C_0402_1005Metric
- C614: renamed from C121; footprint (none) -> Capacitor_SMD:C_0402_1005Metric
- C615: renamed from C132; footprint (none) -> Capacitor_SMD:C_0402_1005Metric
- C616: renamed from C153; footprint (none) -> Capacitor_SMD:C_0402_1005Metric
- C617: renamed from C169; value 100nF -> 1uF; footprint (none) -> Capacitor_SMD:C_0402_1005Metric
- C618: renamed from C167; footprint (none) -> Capacitor_SMD:C_0402_1005Metric
- C619: renamed from C173; footprint (none) -> Capacitor_SMD:C_0402_1005Metric
- C620: renamed from C170; footprint (none) -> Capacitor_SMD:C_0402_1005Metric
- C621: renamed from C177; footprint (none) -> Capacitor_SMD:C_0402_1005Metric
- C622: renamed from C181; footprint (none) -> Capacitor_SMD:C_0402_1005Metric
- C623: renamed from C68; footprint (none) -> Capacitor_SMD:C_0402_1005Metric
- C624: renamed from C75; footprint (none) -> Capacitor_SMD:C_0402_1005Metric
- C625: renamed from C89; footprint (none) -> Capacitor_SMD:C_0402_1005Metric
- C626: renamed from C92; footprint (none) -> Capacitor_SMD:C_0402_1005Metric
- C627: renamed from C185; footprint (none) -> Capacitor_SMD:C_0402_1005Metric
- C628: renamed from C189; footprint (none) -> Capacitor_SMD:C_0402_1005Metric
- R601: renamed from R21; footprint (none) -> Resistor_SMD:R_0402_1005Metric
- R602: renamed from R28; footprint (none) -> Resistor_SMD:R_0402_1005Metric
- R603: renamed from R23; footprint (none) -> Resistor_SMD:R_0402_1005Metric
- R604: renamed from R20; footprint (none) -> Resistor_SMD:R_0402_1005Metric
- R605: renamed from R14; footprint (none) -> Resistor_SMD:R_0402_1005Metric
- R606: renamed from R25; footprint (none) -> Resistor_SMD:R_0402_1005Metric
- R607: renamed from R30; footprint (none) -> Resistor_SMD:R_0402_1005Metric
- R608: renamed from R38; footprint (none) -> Resistor_SMD:R_0402_1005Metric
- R609: renamed from R99; footprint (none) -> Resistor_SMD:R_0402_1005Metric
- U601: renamed from U7; footprint CP_72_5_ADI -> AD8285WBCPZ:CP_72_5_ADI
- renumbered D13 to D601, D9 to D602, D5 to D603, D1 to D604
