File: TX.kicad_sch (KiCad schematic)
At the start: 0 parts

Commit message: finished SOM 5V power, migrated altium stuff, finished pin study, added USB PHY (revise HS capability)
Parts:
- added C1, C2, C3: 1nF, symbol Device:C
- added C17, C18, C27, C28, C29, C30, C31, C32, C33, C34, C35, C36, C37, C38, C39, C40: 1uF 100V, symbol Device:C
- added C19, C20, C21, C22, C23, C24, C25, C26, C41, C42: 100nF, symbol Device:C
- added R1, R2, R3, R4, R5: 10K, symbol Device:R_US
- added U4: (no value), symbol TX7516:TX7516
Connections:
- new net GND: C1.2, C17.2, C18.2, C19.2, C2.2, C20.2, C21.2, C22.2, C23.2, C24.2, C25.2, C26.2, C27.2, C28.2, C29.2, C3.2, C30.2, C31.2, C32.2, C33.2, C34.2, C35.2, C36.2, C37.2, C38.2, C39.2, C40.2, C41.2, C42.2, R2.2, R3.2, R4.2, R5.2, U4.B6 (AVSS), U4.B7 (AVSS), U4.C10 (AVSS), U4.C3 (AVSS), U4.C6 (AVSS), U4.C7 (AVSS), U4.D10 (AVSS), U4.D3 (AVSS), U4.D6 (AVSS), U4.D7 (AVSS), U4.E10 (AVSS), U4.E3 (AVSS), U4.F10 (AVSS), U4.F3 (AVSS), U4.F4 (AVSS), U4.G10 (AVSS), U4.G3 (AVSS), U4.H10 (AVSS), U4.H3 (AVSS), U4.H5 (AVSS), U4.H8 (AVSS), U4.J10 (AVSS), U4.J3 (AVSS), U4.J5 (AVSS), U4.J8 (AVSS), U4.K10 (AVSS), U4.K11 (AVSS), U4.K2 (AVSS), U4.K3 (AVSS), U4.K4 (AVSS), U4.K5 (AVSS), U4.K6 (AVSS), U4.K7 (AVSS), U4.K8 (AVSS), U4.K9 (AVSS), U4.L5 (AVSS), U4.L8 (AVSS), U4.M5 (AVSS), U4.M8 (AVSS)
- new net PULSER_100V: C17.1, C18.1, C27.1, C28.1, C29.1, C30.1, C31.1, C32.1, U4.A4 (AVDDP_HV_A), U4.A5 (AVDDP_HV_B), U4.A8 (AVDDP_HV_B), U4.A9 (AVDDP_HV_A), U4.B4 (AVDDP_HV_A), U4.B5 (AVDDP_HV_B), U4.B8 (AVDDP_HV_B), U4.B9 (AVDDP_HV_A), U4.C4 (AVDDP_HV_A), U4.C5 (AVDDP_HV_B), U4.C8 (AVDDP_HV_B), U4.C9 (AVDDP_HV_A), U4.D4 (AVDDP_HV_A), U4.D5 (AVDDP_HV_B), U4.D8 (AVDDP_HV_B), U4.D9 (AVDDP_HV_A)
- new net PULSER_100VN: C33.1, C34.1, C35.1, C36.1, C37.1, C38.1, C39.1, C40.1, U4.D1 (AVDDM_HV_B), U4.D11 (AVDDM_HV_B), U4.D12 (AVDDM_HV_B), U4.D2 (AVDDM_HV_B), U4.E1 (AVDDM_HV_B), U4.E11 (AVDDM_HV_B), U4.E12 (AVDDM_HV_B), U4.E2 (AVDDM_HV_B), U4.F1 (AVDDM_HV_A), U4.F11 (AVDDM_HV_A), U4.F12 (AVDDM_HV_A), U4.F2 (AVDDM_HV_A), U4.G1 (AVDDM_HV_A), U4.G11 (AVDDM_HV_A), U4.G12 (AVDDM_HV_A), U4.G2 (AVDDM_HV_A)
- new net PULSER_1V8: C41.1, C42.1, R1.1, U4.F8 (AVDDP_1P8), U4.F9 (AVDDP_1P8), U4.G8 (AVDDP_1P8), U4.G9 (AVDDP_1P8)
- new net PULSER_5V: C23.1, C24.1, C25.1, C26.1, U4.E6 (AVDDP_5), U4.E7 (AVDDP_5), U4.E8 (AVDDP_5), U4.E9 (AVDDP_5)
- new net PULSER_5VN: C19.1, C20.1, C21.1, C22.1, U4.E4 (AVDDM_5V), U4.E5 (AVDDM_5V)
- new net PULSER_BF_CLK_N: U4.M6 (BF_CLKM)
- new net PULSER_BF_CLK_P: U4.M7 (BF_CLKP)
- new net PULSER_BF_SYNC_CLK_N: U4.L6 (TR_BF_SYNCM)
- new net PULSER_BF_SYNC_CLK_P: U4.L7 (TR_BF_SYNCP)
- new net PULSER_CRC_ERR: C3.1, R5.1, U4.J2 (CRC_ERR)
- new net PULSER_RESET: U4.J1 (RESET)
- new net PULSER_SPI_CLK_N: U4.J6 (SCLKM)
- new net PULSER_SPI_CLK_P: U4.H6 (SCLKP)
- new net PULSER_SPI_CRC_EN: U4.G4 (EN_CRC)
- new net PULSER_SPI_CS0: U4.F7 (CHIP_SEL0)
- new net PULSER_SPI_CS1: U4.G7 (CHIP_SEL1)
- new net PULSER_SPI_D0_N: R1.2, U4.J7 (SDATAM_1), U4.J9 (SDATAM_0)
- new net PULSER_SPI_D0_P: R2.1, U4.H7 (SDATAP_1), U4.H9 (SDATAP_0)
- new net PULSER_SPI_MODE: U4.G5 (SPI_MODE)
- new net PULSER_SPI_SDOUT: U4.H12 (SDOUT)
- new net PULSER_SPI_SE_N: U4.J4 (SENM)
- new net PULSER_SPI_SE_P: U4.H4 (SENP)
- new net PULSER_TSHUT: C2.1, R4.1, U4.H1 (TSHUT)
- new net PULSER_TXRX: C1.1, R3.1, U4.H11 (TX_RXZ)
- new net PULSER_WAKEUP: U4.J12 (WAKE_UP)
- new net RX_IN1: U4.L12 (RX_1)
- new net RX_IN10: U4.M4 (RX_10)
- new net RX_IN11: U4.L3 (RX_11)
- new net RX_IN12: U4.M3 (RX_12)
- new net RX_IN13: U4.L2 (RX_13)
- new net RX_IN14: U4.M2 (RX_14)
- new net RX_IN15: U4.L1 (RX_15)
- new net RX_IN16: U4.M1 (RX_16)
- new net RX_IN2: U4.M12 (RX_2)
- new net RX_IN3: U4.L11 (RX_3)
- new net RX_IN4: U4.M11 (RX_4)
- new net RX_IN5: U4.L10 (RX_5)
- new net RX_IN6: U4.M10 (RX_6)
- new net RX_IN7: U4.L9 (RX_7)
- new net RX_IN8: U4.M9 (RX_8)
- new net RX_IN9: U4.L4 (RX_9)
- new net TX_OUT1: U4.A12 (OUT_1)
- new net TX_OUT10: U4.B1 (OUT_10)
- new net TX_OUT11: U4.C1 (OUT_11)
- new net TX_OUT12: U4.A2 (OUT_12)
- new net TX_OUT13: U4.B2 (OUT_13)
- new net TX_OUT14: U4.C2 (OUT_14)
- new net TX_OUT15: U4.A3 (OUT_15)
- new net TX_OUT16: U4.B3 (OUT_16)
- new net TX_OUT2: U4.B12 (OUT_2)
- new net TX_OUT3: U4.C12 (OUT_3)
- new net TX_OUT4: U4.A11 (OUT_4)
- new net TX_OUT5: U4.B11 (OUT_5)
- new net TX_OUT6: U4.C11 (OUT_6)
- new net TX_OUT7: U4.A10 (OUT_7)
- new net TX_OUT8: U4.B10 (OUT_8)
- new net TX_OUT9: U4.A1 (OUT_9)
- no-connect marks 0 -> 9

Commit message: added USB (needs revision), fixed medium voltage rail
Parts:
- removed C17, C18, C27, C28, C29, C30, C31, C32: 1uF 100V, symbol Device:C
- added C198, C207, C208, C209, C210, C211, C212, C213: 100nF 200V, symbol Device:C
- C33, C34, C35, C36, C37, C38, C39, C40: value 1uF 100V -> 100nF 200V
Connections:
- net GND: now also C198.2, C207.2, C208.2, C209.2, C210.2, C211.2, C212.2, C213.2
- net PULSER_100V: now also C37.1, C38.1, C39.1, C40.1; no longer U4.A5 (AVDDP_HV_B), U4.A8 (AVDDP_HV_B), U4.B5 (AVDDP_HV_B), U4.B8 (AVDDP_HV_B), U4.C5 (AVDDP_HV_B), U4.C8 (AVDDP_HV_B), U4.D5 (AVDDP_HV_B), U4.D8 (AVDDP_HV_B)
- net PULSER_100VN: no longer C37.1, C38.1, C39.1, C40.1, U4.D1 (AVDDM_HV_B), U4.D11 (AVDDM_HV_B), U4.D12 (AVDDM_HV_B), U4.D2 (AVDDM_HV_B), U4.E1 (AVDDM_HV_B), U4.E11 (AVDDM_HV_B), U4.E12 (AVDDM_HV_B), U4.E2 (AVDDM_HV_B)
- new net PULSER_50V: C198.1, C207.1, C208.1, C209.1, U4.A5 (AVDDP_HV_B), U4.A8 (AVDDP_HV_B), U4.B5 (AVDDP_HV_B), U4.B8 (AVDDP_HV_B), U4.C5 (AVDDP_HV_B), U4.C8 (AVDDP_HV_B), U4.D5 (AVDDP_HV_B), U4.D8 (AVDDP_HV_B)
- new net PULSER_50VN: C210.1, C211.1, C212.1, C213.1, U4.D1 (AVDDM_HV_B), U4.D11 (AVDDM_HV_B), U4.D12 (AVDDM_HV_B), U4.D2 (AVDDM_HV_B), U4.E1 (AVDDM_HV_B), U4.E11 (AVDDM_HV_B), U4.E12 (AVDDM_HV_B), U4.E2 (AVDDM_HV_B)

Commit message: almost finished, phew! just dd +/- 5v rails, connect the SDIO & power enable pins and figure out the rest of the clocking chain
Connections:
- net PULSER_SPI_D0_N: no longer R1.2, U4.J7 (SDATAM_1)
- net PULSER_SPI_D0_P: no longer R2.1, U4.H7 (SDATAP_1)
- net RX_IN1 renamed TR_OUT0
- net RX_IN10 renamed TR_OUT9
- net RX_IN11 renamed TR_OUT10
- net RX_IN12 renamed TR_OUT11
- net RX_IN13 renamed TR_OUT12
- net RX_IN14 renamed TR_OUT13
- net RX_IN15 renamed TR_OUT14
- net RX_IN16 renamed TR_OUT15
- net RX_IN2 renamed TR_OUT1
- net RX_IN3 renamed TR_OUT2
- net RX_IN4 renamed TR_OUT3
- net RX_IN5 renamed TR_OUT4
- net RX_IN6 renamed TR_OUT5
- net RX_IN7 renamed TR_OUT6
- net RX_IN8 renamed TR_OUT7
- net RX_IN9 renamed TR_OUT8
- net TX_OUT1 renamed PULSER_OUT0
- net TX_OUT10 renamed PULSER_OUT9
- net TX_OUT11 renamed PULSER_OUT10
- net TX_OUT12 renamed PULSER_OUT11
- net TX_OUT13 renamed PULSER_OUT12
- net TX_OUT14 renamed PULSER_OUT13
- net TX_OUT15 renamed PULSER_OUT14
- net TX_OUT16 renamed PULSER_OUT15
- net TX_OUT2 renamed PULSER_OUT1
- net TX_OUT3 renamed PULSER_OUT2
- net TX_OUT4 renamed PULSER_OUT3
- net TX_OUT5 renamed PULSER_OUT4
- net TX_OUT6 renamed PULSER_OUT5
- net TX_OUT7 renamed PULSER_OUT6
- net TX_OUT8 renamed PULSER_OUT7
- net TX_OUT9 renamed PULSER_OUT8
- new net PULSER_SPI_D1_N: R1.2, U4.J7 (SDATAM_1)
- new net PULSER_SPI_D1_P: R2.1, U4.H7 (SDATAP_1)

Commit message: HDMI was requested so add it and give the signal chain a final revision
Parts:
- added R15, R16: 10K, symbol Device:R_US
Connections:
- net GND: now also R15.2, R16.2
- net PULSER_RESET: now also R15.1
- net PULSER_WAKEUP: now also R16.1

Commit message: ALL IS DONE EXCEPT HDMI PLEASE HELP
Parts:
- R1, R2: now not fitted; now left out of the parts list
Other:
- note added: "+100V HV Supply"
- note added: "+50V HV Supply"
- note added: "-100V HV Supply"
- note added: "-50V HV Supply"
- note added: "-5V"
- note added: "1.8V"
- note added: "HV Pulser Outputs"
- note added: "Logic 5V"
- note added: "Only place resistors R1 & R2 if data line 1 is not used."
- note added: "Output: Indicates whether the pulser is in transmit or receiver mode."
- note added: "Output: SPI error flag (CRC error)."
- note added: "Output: Thermal shutdown flag."
- note added: "T/R Switch Outputs"
Changed lines of the file:
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@@
 	(generator_version "10.0")
 	(paper "A3")
+	(text "-50V HV Supply"
+		(exclude_from_sim no)
+		(at 254.254 97.79 0)
+		(effects
+			(font
+				(size 3 3)
+				(thickness 0.6)
+				(bold yes)
+			)
+		)
+	)
+	(text "-5V"
+		(exclude_from_sim no)
+		(at 244.856 47.498 0)
+		(effects
+			(font
+				(size 3 3)
+				(thickness 0.6)
+				(bold yes)
+			)
+		)
+	)
+	(text "1.8V"
+		(exclude_from_sim no)
+		(at 244.856 53.848 0)
+		(effects
+			(font
+				(size 3 3)
+				(thickness 0.6)
+				(bold yes)
+			)
+		)
+	)
+	(text "+100V HV Supply"
+		(exclude_from_sim no)
+		(at 253.746 119.888 0)
+		(effects
+			(font
+				(size 3 3)
+				(thickness 0.6)
+				(bold yes)
+			)
+		)
+	)
+	(text "Logic 5V"
+		(exclude_from_sim no)
+		(at 262.382 36.576 0)
+		(effects
+			(font
+				(size 3 3)
+				(thickness 0.6)
+				(bold yes)
+			)
+		)
+	)
+	(text "HV Pulser Outputs"
+		(exclude_from_sim no)
+		(at 205.232 59.944 0)
+		(effects
+			(font
+				(size 3 3)
+				(thickness 0.6)
+				(bold yes)
+			)
+		)
+	)
+	(text "Only place resistors R1 & R2 if data line 1\nis not used."
+		(exclude_from_sim no)
+		(at 15.24 62.23 0)
+		(effects
+			(font
+				(size 1.27 1.27)
+			)
+			(justify left)
+		)
+	)
+	(text "Output:\nIndicates whether the pulser is in\ntransmit or receiver mode."
+		(exclude_from_sim no)
+		(at 28.194 165.862 0)
+		(effects
+			(font
+				(size 1.27 1.27)
+			)
+			(justify left)
+		)
+	)
+	(text "Output:\nSPI error flag (CRC error)."
+		(exclude_from_sim no)
+		(at 118.872 183.388 0)
+		(effects
+			(font
+				(size 1.27 1.27)
+			)
+			(justify left)
+		)
+	)
+	(text "-100V HV Supply"
+		(exclude_from_sim no)
+		(at 253.238 73.406 0)
+		(effects
+			(font
+				(size 3 3)
+				(thickness 0.6)
+				(bold yes)
+			)
+		)
+	)
+	(text "+50V HV Supply"
+		(exclude_from_sim no)
+		(at 254.762 144.272 0)
+		(effects
+			(font
+				(size 3 3)
+				(thickness 0.6)
+				(bold yes)
+			)
+		)
+	)
+	(text "Output:\nThermal shutdown flag."
+		(exclude_from_sim no)
+		(at 84.582 189.738 0)
+		(effects
+			(font
+				(size 1.27 1.27)
+			)
+			(justify left)
+		)
+	)
+	(text "T/R Switch Outputs"
+		(exclude_from_sim no)
+		(at 204.724 102.108 0)
+		(effects
+			(font
+				(size 3 3)
+				(thickness 0.6)
+				(bold yes)
+			)
+		)
+	)
 	(junction
 		(at 279.4 99.06)
@@
 		(body_style 1)
 		(exclude_from_sim no)
-		(in_bom yes)
+		(in_bom no)
 		(on_board yes)
-		(in_pos_files yes)
-		(dnp no)
+		(in_pos_files no)
+		(dnp yes)
 		(property "Reference" "R1"
 			(at 60.96 55.8799 0)
@@
 		(body_style 1)
 		(exclude_from_sim no)
-		(in_bom yes)
+		(in_bom no)
 		(on_board yes)
-		(in_pos_files yes)
-		(dnp no)
+		(in_pos_files no)
+		(dnp yes)
 		(property "Reference" "R2"
 			(at 63.5 69.8499 0)

Commit message: started layout, finished 90% of individual section placement, need to finish remaining and integrate together in PCB and apply schematic edits before
Parts:
- C201: renamed from C1; footprint (none) -> Capacitor_SMD:C_0402_1005Metric
- C202: renamed from C2; footprint (none) -> Capacitor_SMD:C_0402_1005Metric
- C203: renamed from C3; footprint (none) -> Capacitor_SMD:C_0402_1005Metric
- C204: renamed from C37; footprint (none) -> Capacitor_SMD:C_0805_2012Metric
- C205: renamed from C33; footprint (none) -> Capacitor_SMD:C_0805_2012Metric
- C206: renamed from C23; footprint (none) -> Capacitor_SMD:C_0402_1005Metric
- C207: renamed from C41; footprint (none) -> Capacitor_SMD:C_0402_1005Metric
- C208: renamed from C42; footprint (none) -> Capacitor_SMD:C_0402_1005Metric
- C209: renamed from C38; footprint (none) -> Capacitor_SMD:C_0805_2012Metric
- C210: renamed from C34; footprint (none) -> Capacitor_SMD:C_0805_2012Metric
- C211: renamed from C24; footprint (none) -> Capacitor_SMD:C_0402_1005Metric
- C212: renamed from C39; footprint (none) -> Capacitor_SMD:C_0805_2012Metric
- C213: renamed from C35; footprint (none) -> Capacitor_SMD:C_0805_2012Metric
- C214: renamed from C25; footprint (none) -> Capacitor_SMD:C_0402_1005Metric
- C215: renamed from C40; footprint (none) -> Capacitor_SMD:C_0805_2012Metric
- C216: renamed from C36; footprint (none) -> Capacitor_SMD:C_0805_2012Metric
- C217: renamed from C26; footprint (none) -> Capacitor_SMD:C_0402_1005Metric
- C218: renamed from C198; footprint (none) -> Capacitor_SMD:C_0805_2012Metric
- C219: renamed from C210; footprint (none) -> Capacitor_SMD:C_0805_2012Metric
- C220: renamed from C21; footprint (none) -> Capacitor_SMD:C_0402_1005Metric
- C221: renamed from C207; footprint (none) -> Capacitor_SMD:C_0805_2012Metric
- C222: renamed from C211; footprint (none) -> Capacitor_SMD:C_0805_2012Metric
- C223: renamed from C22; footprint (none) -> Capacitor_SMD:C_0402_1005Metric
- C224: renamed from C208; footprint (none) -> Capacitor_SMD:C_0805_2012Metric
- C225: renamed from C212; footprint (none) -> Capacitor_SMD:C_0805_2012Metric
- C226: renamed from C20; footprint (none) -> Capacitor_SMD:C_0402_1005Metric
- C227: renamed from C209; footprint (none) -> Capacitor_SMD:C_0805_2012Metric
- C228: renamed from C213; footprint (none) -> Capacitor_SMD:C_0805_2012Metric
- C229: renamed from C19; footprint (none) -> Capacitor_SMD:C_0402_1005Metric
- R201: renamed from R15; footprint (none) -> Resistor_SMD:R_0402_1005Metric
- R202: renamed from R1; footprint (none) -> Resistor_SMD:R_0402_1005Metric
- R203: renamed from R16; footprint (none) -> Resistor_SMD:R_0402_1005Metric
- R204: renamed from R3; footprint (none) -> Resistor_SMD:R_0402_1005Metric
- R205: renamed from R2; footprint (none) -> Resistor_SMD:R_0402_1005Metric
- R206: renamed from R4; footprint (none) -> Resistor_SMD:R_0402_1005Metric
- R207: renamed from R5; footprint (none) -> Resistor_SMD:R_0402_1005Metric
- U201: renamed from U4; footprint (none) -> TX7516:BGA-144_10.0x10.0mm_Layout12x12_P0.8mm_TI-ALH0144A
