File: 100V_Supply.kicad_sch (KiCad schematic)
At the start: 26 parts, among them Q1 FDMC86240, U1 LM5155DSSR

Commit message: ALL IS DONE EXCEPT HDMI PLEASE HELP
Parts:
- added JP14: 100V_JMP, Package_LCC:PLCC-84_29.3x29.3mm_P1.27mm, symbol Jumper:SolderJumper_2_Open
- added JP15: -100V_JMP, Package_LCC:PLCC-84_29.3x29.3mm_P1.27mm, symbol Jumper:SolderJumper_2_Open
Connections:
- net PULSER_100V: now also JP14.2 (B); no longer C56.1, L8.2
- net PULSER_100VN: now also JP15.2 (B); no longer C59.2, L7.2
- new net PULSER_100VN_PRE: C59.2, JP15.1 (A), L7.2
- new net PULSER_100V_PRE: C56.1, JP14.1 (A), L8.2

Commit message: started layout, finished 90% of individual section placement, need to finish remaining and integrate together in PCB and apply schematic edits before
Parts:
- C1601: renamed from C60; footprint (none) -> Capacitor_SMD:C_0805_2012Metric
- C1602: renamed from C14; footprint (none) -> Capacitor_SMD:C_0805_2012Metric
- C1603: renamed from C194; footprint (none) -> Capacitor_SMD:C_0402_1005Metric
- C1604: renamed from C61; footprint (none) -> Capacitor_SMD:C_0402_1005Metric
- C1605: renamed from C193; footprint (none) -> Capacitor_SMD:C_0402_1005Metric
- C1606: renamed from C52; footprint (none) -> Capacitor_SMD:C_0805_2012Metric
- C1607: renamed from C53; footprint (none) -> Capacitor_SMD:C_0805_2012Metric
- C1608: renamed from C55; footprint (none) -> Capacitor_SMD:C_1812_4532Metric
- C1609: renamed from C57; footprint (none) -> Capacitor_SMD:C_1812_4532Metric
- C1610: renamed from C56; footprint (none) -> Capacitor_SMD:C_1812_4532Metric
- C1611: renamed from C59; footprint (none) -> Capacitor_SMD:C_1812_4532Metric
- JP1601: renamed from JP14; footprint Package_LCC:PLCC-84_29.3x29.3mm_P1.27mm -> Jumper:SolderJumper-2_P1.3mm_Open_TrianglePad1.0x1.5mm
- JP1602: renamed from JP15; footprint Package_LCC:PLCC-84_29.3x29.3mm_P1.27mm -> Jumper:SolderJumper-2_P1.3mm_Open_TrianglePad1.0x1.5mm
- L1601: renamed from L5; footprint (none) -> Inductor_SMD:L_Panasonic_PCC-M0854M
- L1602: renamed from L4; footprint (none) -> Inductor_SMD:L_Cenker_CKCS4018
- L1603: renamed from L6; footprint (none) -> Inductor_SMD:L_Cenker_CKCS4018
- L1604: renamed from L8; footprint (none) -> Inductor_SMD:L_Cenker_CKCS4018
- L1605: renamed from L7; footprint (none) -> Inductor_SMD:L_Cenker_CKCS4018
- Q1601: renamed from Q1; footprint FDMC86139P -> FDMC86240:FDMC86139P
- R1601: renamed from R58; footprint (none) -> Resistor_SMD:R_0402_1005Metric
- R1602: renamed from R48; footprint (none) -> Resistor_SMD:R_0402_1005Metric
- R1603: renamed from R47; footprint (none) -> Resistor_SMD:R_0402_1005Metric
- R1604: renamed from R49; footprint (none) -> Resistor_SMD:R_0603_1608Metric
- R1605: renamed from R50; footprint (none) -> Resistor_SMD:R_0402_1005Metric
- R1606: renamed from R51; footprint (none) -> Resistor_SMD:R_0402_1005Metric
- renumbered D17 to D1601, D18 to D1602, U1 to U1601

Commit message: finished preliminary placement, will definietly be changed when routing don't forget to apply comments in first page and calculate trace impedance for all traces & make AI revise schematic
Connections:
- net PULSER_100V: no longer R1605.1
- net PULSER_100V_PRE: now also R1605.1
