File: 50V_Supply.kicad_sch (KiCad schematic)
At the start: 26 parts, among them Q2 FDMC86240, U2 LM5155DSSR

Commit message: ALL IS DONE EXCEPT HDMI PLEASE HELP
Parts:
- added JP17: -50V_JMP, symbol Jumper:SolderJumper_2_Open
- added JP18: 50V_JMP, symbol Jumper:SolderJumper_2_Open
Connections:
- net PULSER_50V: now also JP18.2 (B); no longer C204.1, L12.2
- net PULSER_50VN: now also JP17.2 (B); no longer C205.2, L13.2
- new net PULSER_50VN_PRE: C205.2, JP17.1 (A), L13.2
- new net PULSER_50V_PRE: C204.1, JP18.1 (A), L12.2

Commit message: started layout, finished 90% of individual section placement, need to finish remaining and integrate together in PCB and apply schematic edits before
Parts:
- C1401: renamed from C195; footprint (none) -> Capacitor_SMD:C_0805_2012Metric
- C1402: renamed from C196; footprint (none) -> Capacitor_SMD:C_0805_2012Metric
- C1403: renamed from C197; footprint (none) -> Capacitor_SMD:C_0402_1005Metric
- C1404: renamed from C206; footprint (none) -> Capacitor_SMD:C_0402_1005Metric
- C1405: renamed from C199; footprint (none) -> Capacitor_SMD:C_0402_1005Metric
- C1406: renamed from C200; footprint (none) -> Capacitor_SMD:C_0805_2012Metric
- C1407: renamed from C201; footprint (none) -> Capacitor_SMD:C_0805_2012Metric
- C1408: renamed from C202; footprint (none) -> Capacitor_SMD:C_1812_4532Metric
- C1409: renamed from C203; footprint (none) -> Capacitor_SMD:C_1812_4532Metric
- C1410: renamed from C204; footprint (none) -> Capacitor_SMD:C_1812_4532Metric
- C1411: renamed from C205; footprint (none) -> Capacitor_SMD:C_1812_4532Metric
- JP1401: renamed from JP18; footprint (none) -> Jumper:SolderJumper-2_P1.3mm_Open_TrianglePad1.0x1.5mm
- JP1402: renamed from JP17; footprint (none) -> Jumper:SolderJumper-2_P1.3mm_Open_TrianglePad1.0x1.5mm
- L1401: renamed from L9; footprint (none) -> Inductor_SMD:L_SXN_SMDRI127
- L1402: renamed from L10; footprint (none) -> Inductor_SMD:L_Cenker_CKCS4018
- L1403: renamed from L11; footprint (none) -> Inductor_SMD:L_Cenker_CKCS4018
- L1404: renamed from L12; footprint (none) -> Inductor_SMD:L_1210_3225Metric
- L1405: renamed from L13; footprint (none) -> Inductor_SMD:L_1210_3225Metric
- Q1401: renamed from Q2; footprint FDMC86139P -> FDMC86240:FDMC86139P
- R1401: renamed from R59; footprint (none) -> Resistor_SMD:R_0402_1005Metric
- R1402: renamed from R52; footprint (none) -> Resistor_SMD:R_0402_1005Metric
- R1403: renamed from R53; footprint (none) -> Resistor_SMD:R_0402_1005Metric
- R1404: renamed from R54; footprint (none) -> Resistor_SMD:R_0603_1608Metric
- R1405: renamed from R55; footprint (none) -> Resistor_SMD:R_0402_1005Metric
- R1406: renamed from R56; footprint (none) -> Resistor_SMD:R_0402_1005Metric
- renumbered D19 to D1401, D20 to D1402, U2 to U1401

Commit message: finished preliminary placement, will definietly be changed when routing don't forget to apply comments in first page and calculate trace impedance for all traces & make AI revise schematic
Connections:
- net PULSER_100V is gone; now on net PULSER_50V_PRE: R1405.1
Changed lines of the file:
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@@
 		(dnp no)
 		(fields_autoplaced yes)
-		(property "Reference" "#PWR01408"
+		(property "Reference" "#PWR01416"
 			(at 171.45 124.46 0)
 			(hide yes)
@@
 			)
 		)
-		(property "Value" "PULSER_100V"
+		(property "Value" "PULSER_50V_PRE"
 			(at 171.45 115.57 0)
 			(show_name no)
@@
 			)
 		)
-		(property "Description" "Power symbol creates a global label with name \"PULSER_100V\""
+		(property "Description" "Power symbol creates a global label with name \"PULSER_50V_PRE\""
 			(at 171.45 120.65 0)
 			(hide yes)
@@
 			(project "MedicalImager"
 				(path "/99848109-7be9-4113-bc9c-faf6c2acfe0b/bd63d6e1-5dfb-4921-86f2-9a66ea07210d/e269633f-c26a-42b5-a12c-87dd41533928"
-					(reference "#PWR01408")
+					(reference "#PWR01416")
 					(unit 1)
 				)
