File: Interface.kicad_sch (KiCad schematic)
At the start: 60 parts, among them J3 47352-1001, J4 2086581001, J5 External Board 2, J6 External Board 1, J7 TYPE-C-31-M-12, U10 USBLC6-2SC6, U13 TUSB1210BRHBR, U18 SN75DP139RSBR, U24 NVT4858HKZ, U9 NXB0108BQ-Q100X

Commit message: started layout, finished 90% of individual section placement, need to finish remaining and integrate together in PCB and apply schematic edits before
Parts:
- removed C246, C247, C248, C249, C250, C251, C252, C253, C254, C255, C256, C257, C258, C259, C260, C261: 100nF, symbol Device:C
- removed CR1: DT1240A-08LP3810-7, U-DFN3810-9_TYPE_B_DIO, symbol DT1240A-08LP3810-7:DT1240A-08LP3810-7
- removed J4: 2086581001, 2086581001:MOLEX_2086581001, symbol 2086581001:2086581001
- removed JP16: HPD_INV_PUP, U-DFN3810-9_TYPE_B_DIO, symbol Jumper:SolderJumper_2_Open
- removed R106, R107, R67, R68, R85, R86, R87, R88: 10K, symbol Device:R_US
- removed R17: 4.02K, symbol Device:R_US
- removed R69, R70, R83, R84: 3.3k, symbol Device:R_US
- removed U18: SN75DP139RSBR, RSB40_3P15X3P15, symbol SN75DP139RSBR:SN75DP139RSBR
- added C1001: 47uF, Capacitor_SMD:C_0805_2012Metric, symbol Device:C
- added C1002: 100nF, Capacitor_SMD:C_0805_2012Metric, symbol Device:C
- added C1004, C1008: 100nF, Capacitor_SMD:C_0402_1005Metric, symbol Device:C
- added F1001: 0154.500DRT, 0154-500DRT:0154Series_LTF, symbol 0154-500DRT:0154.500DRT
- added J1002: B8B-XH-A, B8B-XH-A:JST_B8B-XH-A, symbol B8B-XH-A:B8B-XH-A
- added Q1001: SI2302DS, SI2302DS:SOT23-3_TO-236AB, symbol SI2302DS:SI2302DS
- added R1004, R1005: 10K, Resistor_SMD:R_0402_1005Metric, symbol Device:R_US
- added U1004: NXB0104PWJ, NXB0104PWJ:SOP65P640X120-14N, symbol NXB0104PWJ:NXB0104PWJ
- C1003: renamed from C240; footprint (none) -> Capacitor_SMD:C_0402_1005Metric
- C1005: renamed from C47; footprint (none) -> Capacitor_SMD:C_0805_2012Metric
- C1006: renamed from C241; footprint (none) -> Capacitor_SMD:C_0402_1005Metric
- C1007: renamed from C227; footprint (none) -> Capacitor_SMD:C_0402_1005Metric
- C1009: renamed from C228; footprint (none) -> Capacitor_SMD:C_0402_1005Metric
- C1010: renamed from C226; footprint (none) -> Capacitor_SMD:C_0402_1005Metric
- C1011: renamed from C242; footprint (none) -> Capacitor_SMD:C_0402_1005Metric
- C1012: renamed from C214; footprint (none) -> Capacitor_SMD:C_0402_1005Metric
- C1013: renamed from C243; footprint (none) -> Capacitor_SMD:C_0402_1005Metric
- C1014: renamed from C216; footprint (none) -> Capacitor_SMD:C_0402_1005Metric
- C1015: renamed from C217; footprint (none) -> Capacitor_SMD:C_0402_1005Metric
- C1016: renamed from C165; footprint (none) -> Capacitor_SMD:C_0402_1005Metric
- C1017: renamed from C164; footprint (none) -> Capacitor_SMD:C_0402_1005Metric
- C1018: renamed from C166; footprint (none) -> Capacitor_SMD:C_0402_1005Metric
- J1003: renamed from J6; footprint (none) -> Connector_PinHeader_2.54mm:PinHeader_2x06_P2.54mm_Vertical
- J1004: renamed from J5; footprint (none) -> Connector_PinHeader_2.54mm:PinHeader_2x06_P2.54mm_Vertical
- R1001: renamed from R110; footprint (none) -> Resistor_SMD:R_0402_1005Metric
- R1002: renamed from R111; footprint (none) -> Resistor_SMD:R_0402_1005Metric
- R1003: renamed from R61; footprint (none) -> Resistor_SMD:R_0402_1005Metric
- R1006: renamed from R109; footprint (none) -> Resistor_SMD:R_0402_1005Metric
- R1007: renamed from R65; footprint (none) -> Resistor_SMD:R_0402_1005Metric
- U1001: renamed from U9; footprint DHVQFN20_SOT764-1_NEX -> NXB0108BQ-Q100X:DHVQFN20_SOT764-1_NEX
- U1003: renamed from U13; footprint RHB32_3P45X3P45 -> TUSB1210BRHBR:RHB32_3P45X3P45
- U1005: renamed from U24; footprint NVT4858_NXP -> NVT4858HKZ:NVT4858_NXP
- renumbered J7 to J1001, J3 to J1005, U10 to U1002
Connections:
- net GND: now also C1001.2, C1002.1, C1004.1, C1008.1, Q1001.2, R1005.2, U1004.7 (GND)
- net SD_DAT0: now also U1005.2 (DAT3A); no longer U1005.3 (DAT0A)
- net SD_DAT0_PRE: now also U1005.11 (DAT3B); no longer U1005.10 (DAT0B)
- net SD_DAT1: now also U1005.1 (DAT2A); no longer U1005.4 (DAT1A)
- net SD_DAT1_PRE: now also U1005.12 (DAT2B); no longer U1005.9 (DAT1B)
- net SD_DAT2: now also U1005.4 (DAT1A); no longer U1005.1 (DAT2A)
- net SD_DAT2_PRE: now also U1005.9 (DAT1B); no longer U1005.12 (DAT2B)
- net SD_DAT3: now also U1005.3 (DAT0A); no longer U1005.2 (DAT3A)
- net SD_DAT3_PRE: now also U1005.10 (DAT0B); no longer U1005.11 (DAT3B)
- net VDD_HPA: now also C1004.2, U1004.1 (VCC_A), U1004.8 (OE)
- net EXT_AFE_CS1_1V8 renamed EXT_AFE_CS1_3V3
- net EXT_AFE_CS2_1V8 renamed EXT_AFE_CS2_3V3
- net EXT_MISO_1V8 renamed EXT_MISO_3V3
- net EXT_MOSI_1V8 renamed EXT_MOSI_3V3
- net EXT_MUX_CS1_1V8 renamed EXT_MUX_CS1_3V3
- net EXT_MUX_CS2_1V8 renamed EXT_MUX_CS2_3V3
- net EXT_RESET_1V8 renamed EXT_RESET_3V3
- net EXT_SCLK_1V8 renamed EXT_SCLK_3V3
- new net: J1002.7, J1002.8, Q1001.3
- new net DC_MAIN: F1001.1
- new net IM_5V: C1008.2, U1004.14 (VCC_B)
- new net LCD_POWER: R1004.2
- new net LCD_POWER_GATE: Q1001.1, R1004.1, R1005.1
- new net LCD_RX2: J1002.5, U1004.11 (B3)
- new net LCD_RX4: J1002.6, U1004.10 (B4)
- new net LCD_RX_AUX: U1004.5 (A4)
- new net LCD_RX_MAIN: U1004.4 (A3)
- new net LCD_TX2: J1002.4, U1004.12 (B2)
- new net LCD_TX4: J1002.3, U1004.13 (B1)
- new net LCD_TX_AUX: U1004.2 (A1)
- new net LCD_TX_MAIN: U1004.3 (A2)
- new net LCD_VCC: C1001.1, C1002.2, F1001.2, J1002.1, J1002.2
- no-connect marks 10 -> 11
Other:
- removed sheet DP2HDMI
- note added: "A slow-blow fuse is used to ignore surges above 0.5A (which should ideally never occur)"
- note added: "Display"

Commit message: finished preliminary placement, will definietly be changed when routing don't forget to apply comments in first page and calculate trace impedance for all traces & make AI revise schematic
Parts:
- added C1019: 100nF, Capacitor_SMD:C_0402_1005Metric, symbol Device:C
- added R1008: 50R, Resistor_SMD:R_0402_1005Metric, symbol Device:R_US
- added Y1001: TG-5006CG-12H_26.0000M3, TG-5006CG-12H 26.0000M3:TG5006CG12H260000M3, symbol TG-5006CG-12H_26_0000M3:TG-5006CG-12H_26.0000M3
Connections:
- net GND: now also C1019.1, Y1001.2 (GND); no longer U1003.1 (REFCLK)
- net USB_PRE_N: now also U1003.18 (DP); no longer U1003.19 (DM)
- net USB_PRE_P: now also U1003.19 (DM); no longer U1003.18 (DP)
- net USB_CLK renamed USB_SOM_CLK
- new net CLK_3V3: C1019.2, Y1001.4 (VCC)
- new net USB_REFCLK: R1008.1, U1003.1 (REFCLK)
- new net USB_REFCLK_PRE: R1008.2, Y1001.3 (OUT)
- no-connect marks 11 -> 12
Other:
- moved on the sheet: R1003, U1002
