File: MedicalImager.kicad_sch (KiCad schematic)
At the start: 0 parts

Commit message: finished preliminary placement, will definietly be changed when routing don't forget to apply comments in first page and calculate trace impedance for all traces & make AI revise schematic
Connections:
- no-connect marks 1 -> 4
Other:
- sheet Interface ports: added LCD_POWER; removed none
- sheet SOM ports: added LCD_POWER, LCD_RX_AUX, LCD_RX_MAIN, LCD_TX_AUX, LCD_TX_MAIN; removed CLK_1V8_EN, CLK_PWR_EN, SOM_5V_PG
- note added: "TODO: - DETAIL THE INDUCTORS' FOOTPRINTS AT THE END - ENSURE STRAPPING RESISTORS ARE AT ALL CS/EN PINS - Add LEDs at all unconnected PG signals"
- note removed: "TODO: - DETAIL THE INDUCTORS' FOOTPRINTS AT THE END - ENSURE STRAPPING RESISTORS ARE AT ALL CS/EN PINS"
Changed lines of the file:
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@@
 	(generator_version "10.0")
 	(paper "A3")
-	(text "TODO:\n- DETAIL THE INDUCTORS' FOOTPRINTS AT THE END\n- ENSURE STRAPPING RESISTORS ARE AT ALL CS/EN PINS"
+	(text "TODO:\n- DETAIL THE INDUCTORS' FOOTPRINTS AT THE END\n- ENSURE STRAPPING RESISTORS ARE AT ALL CS/EN PINS\n- Add LEDs at all unconnected PG signals"
 		(exclude_from_sim no)
-		(at 119.126 211.836 0)
+		(at 98.044 199.39 0)
 		(effects
 			(font
@@
 	)
 	(no_connect
+		(at 127 38.1)
+	)
+	(no_connect
+		(at 86.36 38.1)
+	)
+	(no_connect
+		(at 96.52 38.1)
+	)
+	(no_connect
 		(at 78.74 44.45)
 	)
@@
 	(wire
 		(pts
-			(xy 96.52 38.1) (xy 96.52 44.45)
-		)
-		(stroke
-			(width 0)
-			(type default)
-		)
-	)
-	(wire
-		(pts
 			(xy 50.8 90.17) (xy 63.5 90.17)
 		)
@@
 	(wire
 		(pts
-			(xy 86.36 38.1) (xy 86.36 44.45)
-		)
-		(stroke
-			(width 0)
-			(type default)
-		)
-	)
-	(wire
-		(pts
 			(xy 50.8 77.47) (xy 63.5 77.47)
 		)
@@
 	(wire
 		(pts
+			(xy 50.8 133.35) (xy 63.5 133.35)
+		)
+		(stroke
+			(width 0)
+			(type default)
+		)
+	)
+	(wire
+		(pts
 			(xy 165.1 100.33) (xy 177.8 100.33)
 		)
@@
 	(wire
 		(pts
+			(xy 50.8 138.43) (xy 63.5 138.43)
+		)
+		(stroke
+			(width 0)
+			(type default)
+		)
+	)
+	(wire
+		(pts
 			(xy 119.38 38.1) (xy 119.38 44.45)
 		)
@@
 	(wire
 		(pts
+			(xy 50.8 135.89) (xy 63.5 135.89)
+		)
+		(stroke
+			(width 0)
+			(type default)
+		)
+	)
+	(wire
+		(pts
 			(xy 50.8 113.03) (xy 63.5 113.03)
 		)
@@
 	(wire
 		(pts
+			(xy 50.8 143.51) (xy 63.5 143.51)
+		)
+		(stroke
+			(width 0)
+			(type default)
+		)
+	)
+	(wire
+		(pts
 			(xy 214.63 170.18) (xy 214.63 120.65)
 		)
@@
 	(wire
 		(pts
-			(xy 50.8 54.61) (xy 63.5 54.61)
+			(xy 50.8 140.97) (xy 63.5 140.97)
 		)
 		(stroke
@@
 	(wire
 		(pts
-			(xy 121.92 144.78) (xy 121.92 152.4)
+			(xy 50.8 54.61) (xy 63.5 54.61)
 		)
 		(stroke
@@
 	(wire
 		(pts
-			(xy 109.22 38.1) (xy 109.22 44.45)
+			(xy 121.92 144.78) (xy 121.92 152.4)
 		)
 		(stroke
@@
 	(wire
 		(pts
-			(xy 144.78 144.78) (xy 144.78 152.4)
+			(xy 109.22 38.1) (xy 109.22 44.45)
 		)
 		(stroke
@@
 	(wire
 		(pts
-			(xy 127 38.1) (xy 127 44.45)
+			(xy 144.78 144.78) (xy 144.78 152.4)
 		)
 		(stroke
@@
 			)
 		)
-		(pin "USB_26MHZ" input
+		(pin "USB_26MHZ" bidirectional
 			(at 50.8 77.47 0)
 			(effects
@@
 			)
 		)
+		(pin "LCD_POWER" input
+			(at 50.8 133.35 0)
+			(effects
+				(font
+					(size 1.27 1.27)
+				)
+				(justify right)
+			)
+		)
 		(instances
 			(project "MedicalImager"
@@
 			)
 		)
-		(pin "SOM_5V_PG" input
-			(at 86.36 44.45 90)
-			(effects
-				(font
-					(size 1.27 1.27)
-				)
-				(justify right)
-			)
-		)
 		(pin "50V_EN" output
 			(at 111.76 44.45 90)
@@
 			)
 		)
-		(pin "CLK_PWR_EN" output
-			(at 96.52 44.45 90)
-			(effects
-				(font
-					(size 1.27 1.27)
-				)
-				(justify right)
-			)
-		)
 		(pin "PULSER_SPI_MODE" output
 			(at 165.1 87.63 0)
@@
 			)
 		)
-		(pin "CLK_1V8_EN" output
-			(at 127 44.45 90)
-			(effects
-				(font
-					(size 1.27 1.27)
-				)
-				(justify right)
-			)
-		)
 		(pin "AFE_3V3_EN" output
 			(at 119.38 44.45 90)
@@
 			)
 		)
-		(pin "USB_26MHZ" output
+		(pin "USB_26MHZ" bidirectional
 			(at 63.5 77.47 180)
 			(effects
 				(font
+					(size 1.27 1.27)
+				)
+				(justify left)
+			)
+		)
+		(pin "LCD_TX_AUX" input
+			(at 63.5 140.97 180)
+			(effects
+				(font
+					(size 1.27 1.27)
+				)
+				(justify left)
+			)
+		)
+		(pin "LCD_RX_MAIN" output
+			(at 63.5 138.43 180)
+			(effects
+				(font
+					(size 1.27 1.27)
+				)
+				(justify left)
+			)
+		)
+		(pin "LCD_RX_AUX" output
+			(at 63.5 143.51 180)
+			(effects
+				(font
+					(size 1.27 1.27)
+				)
+				(justify left)
+			)
+		)
+		(pin "LCD_POWER" output
+			(at 63.5 133.35 180)
+			(effects
+				(font
+					(size 1.27 1.27)
+				)
+				(justify left)
+			)
+		)
+		(pin "LCD_TX_MAIN" input
+			(at 63.5 135.89 180)
+			(effects
+				(font
