File: RX.kicad_sch (KiCad schematic)
At the start: 28 parts, among them U301 LMK1D1204RGTR, U302 LMK1D1204RGTR, Y301 ASFLMB-72.000MHZ-LY-T

Commit message: finished preliminary placement, will definietly be changed when routing don't forget to apply comments in first page and calculate trace impedance for all traces & make AI revise schematic
Parts:
- removed C308, C325: 100nF, Capacitor_SMD:C_0402_1005Metric, symbol Device:C
- removed C326: 10uF, Capacitor_SMD:C_0402_1005Metric, symbol Device:C
