File: SOM.kicad_sch (KiCad schematic)
At the start: 29 parts, among them J501 REF-226081-01, J502 REF-226081-01, SW501 RESET

Commit message: finished preliminary placement, will definietly be changed when routing don't forget to apply comments in first page and calculate trace impedance for all traces & make AI revise schematic
Parts:
- SW501: footprint Button_Switch_SMD:Nidec_Copal_CAS-120A -> Button_Switch_SMD:SW_Push_SPST_NO_Alps_SKRK
Connections:
- net AFE_OUTPUTS0: now also J502.D44; no longer J502.B44
- net AFE_OUTPUTS1: now also J502.D45; no longer J502.B45
- net AFE_OUTPUTS10: now also J502.C51; no longer J502.A51
- net AFE_OUTPUTS11: now also J502.C52; no longer J502.A52
- net AFE_OUTPUTS12: now also J502.B44; no longer J502.B52
- net AFE_OUTPUTS13: now also J502.B45; no longer J502.B53
- net AFE_OUTPUTS14: now also J502.B46; no longer J502.B54
- net AFE_OUTPUTS15: now also J502.A46; no longer J502.A54
- net AFE_OUTPUTS16: now also J502.A47; no longer J502.A55
- net AFE_OUTPUTS17: now also J502.A48; no longer J502.A56
- net AFE_OUTPUTS18: now also J502.B48; no longer J502.B56
- net AFE_OUTPUTS19: now also J502.B49; no longer J502.B57
- net AFE_OUTPUTS2: now also J502.D46; no longer J502.B46
- net AFE_OUTPUTS20: now also J502.B50; no longer J502.B58
- net AFE_OUTPUTS21: now also J502.A50; no longer J502.A58
- net AFE_OUTPUTS22: now also J502.A51; no longer J502.A59
- net AFE_OUTPUTS23: now also J502.A52; no longer J502.A60
- net AFE_OUTPUTS24: now also J502.D52; no longer J502.D44
- net AFE_OUTPUTS25: now also J502.D53; no longer J502.D45
- net AFE_OUTPUTS26: now also J502.D54; no longer J502.D46
- net AFE_OUTPUTS27: now also J502.C54; no longer J502.C46
- net AFE_OUTPUTS28: now also J502.C55; no longer J502.C47
- net AFE_OUTPUTS29: now also J502.C56; no longer J502.C48
- net AFE_OUTPUTS3: now also J502.C46; no longer J502.A46
- net AFE_OUTPUTS30: now also J502.D56; no longer J502.D48
- net AFE_OUTPUTS31: now also J502.D57; no longer J502.D49
- net AFE_OUTPUTS32: now also J502.D58; no longer J502.D50
- net AFE_OUTPUTS33: now also J502.C58; no longer J502.C50
- net AFE_OUTPUTS34: now also J502.C59; no longer J502.C51
- net AFE_OUTPUTS35: now also J502.C60; no longer J502.C52
- net AFE_OUTPUTS36: now also J502.B52; no longer J502.D52
- net AFE_OUTPUTS37: now also J502.B53; no longer J502.D53
- net AFE_OUTPUTS38: now also J502.B54; no longer J502.D54
- net AFE_OUTPUTS39: now also J502.A54; no longer J502.C54
- net AFE_OUTPUTS4: now also J502.C47; no longer J502.A47
- net AFE_OUTPUTS40: now also J502.A55; no longer J502.C55
- net AFE_OUTPUTS41: now also J502.A56; no longer J502.C56
- net AFE_OUTPUTS42: now also J502.B56; no longer J502.D56
- net AFE_OUTPUTS43: now also J502.B57; no longer J502.D57
- net AFE_OUTPUTS44: now also J502.B58; no longer J502.D58
- net AFE_OUTPUTS45: now also J502.A58; no longer J502.C58
- net AFE_OUTPUTS46: now also J502.A59; no longer J502.C59
- net AFE_OUTPUTS47: now also J502.A60; no longer J502.C60
- net AFE_OUTPUTS5: now also J502.C48; no longer J502.A48
- net AFE_OUTPUTS6: now also J502.D48; no longer J502.B48
- net AFE_OUTPUTS7: now also J502.D49; no longer J502.B49
- net AFE_OUTPUTS8: now also J502.D50; no longer J502.B50
- net AFE_OUTPUTS9: now also J502.C50; no longer J502.A50
Changed lines of the file:
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@@
 	)
 	(label "AFE_OUTPUTS47"
-		(at 303.53 177.8 0)
+		(at 208.28 177.8 0)
 		(effects
 			(font
@@
 	)
 	(label "AFE_OUTPUTS5"
-		(at 208.28 147.32 0)
+		(at 302.26 147.32 0)
 		(effects
 			(font
@@
 	)
 	(label "AFE_OUTPUTS33"
-		(at 303.53 152.4 0)
+		(at 302.26 172.72 0)
 		(effects
 			(font
@@
 	)
 	(label "AFE_OUTPUTS2"
-		(at 269.24 142.24 180)
+		(at 363.22 142.24 180)
 		(effects
 			(font
@@
 	)
 	(label "AFE_OUTPUTS38"
-		(at 361.95 162.56 180)
+		(at 269.24 162.56 180)
 		(effects
 			(font
@@
 	)
 	(label "AFE_OUTPUTS1"
-		(at 269.24 139.7 180)
+		(at 363.22 139.7 180)
 		(effects
 			(font
@@
 	)
 	(label "AFE_OUTPUTS45"
-		(at 303.53 172.72 0)
+		(at 208.28 172.72 0)
 		(effects
 			(font
@@
 	)
 	(label "AFE_OUTPUTS46"
-		(at 303.53 175.26 0)
+		(at 208.28 175.26 0)
 		(effects
 			(font
@@
 	)
 	(label "AFE_OUTPUTS12"
-		(at 269.24 157.48 180)
+		(at 269.24 137.16 180)
 		(effects
 			(font
@@
 	)
 	(label "AFE_OUTPUTS41"
-		(at 303.53 167.64 0)
+		(at 208.28 167.64 0)
 		(effects
 			(font
@@
 	)
 	(label "AFE_OUTPUTS35"
-		(at 303.53 157.48 0)
+		(at 302.26 177.8 0)
 		(effects
 			(font
@@
 	)
 	(label "AFE_OUTPUTS37"
-		(at 361.95 160.02 180)
+		(at 269.24 160.02 180)
 		(effects
 			(font
@@
 	)
 	(label "AFE_OUTPUTS11"
-		(at 208.28 157.48 0)
+		(at 302.26 157.48 0)
 		(effects
 			(font
@@
 	)
 	(label "AFE_OUTPUTS25"
-		(at 361.95 139.7 180)
+		(at 363.22 160.02 180)
 		(effects
 			(font
@@
 	)
 	(label "AFE_OUTPUTS9"
-		(at 208.28 152.4 0)
+		(at 302.26 152.4 0)
 		(effects
 			(font
@@
 	)
 	(label "AFE_OUTPUTS26"
-		(at 361.95 142.24 180)
+		(at 363.22 162.56 180)
 		(effects
 			(font
@@
 	)
 	(label "AFE_OUTPUTS0"
-		(at 269.24 137.16 180)
+		(at 363.22 137.16 180)
 		(effects
 			(font
@@
 	)
 	(label "AFE_OUTPUTS7"
-		(at 269.24 149.86 180)
+		(at 363.22 149.86 180)
 		(effects
 			(font
@@
 	)
 	(label "AFE_OUTPUTS29"
-		(at 303.53 147.32 0)
+		(at 302.26 167.64 0)
 		(effects
 			(font
@@
 	)
 	(label "AFE_OUTPUTS17"
-		(at 208.28 167.64 0)
+		(at 208.28 147.32 0)
 		(effects
 			(font
@@
 	)
 	(label "AFE_OUTPUTS19"
-		(at 269.24 170.18 180)
+		(at 269.24 149.86 180)
 		(effects
 			(font
@@
 	)
 	(label "AFE_OUTPUTS40"
-		(at 303.53 165.1 0)
+		(at 208.28 165.1 0)
 		(effects
 			(font
@@
 	)
 	(label "AFE_OUTPUTS39"
-		(at 303.53 162.56 0)
+		(at 208.28 162.56 0)
 		(effects
 			(font
@@
 	)
 	(label "AFE_OUTPUTS14"
-		(at 269.24 162.56 180)
+		(at 269.24 142.24 180)
 		(effects
 			(font
@@
 	)
 	(label "AFE_OUTPUTS20"
-		(at 269.24 172.72 180)
+		(at 269.24 152.4 180)
 		(effects
 			(font
@@
 	)
 	(label "AFE_OUTPUTS43"
-		(at 361.95 170.18 180)
+		(at 269.24 170.18 180)
 		(effects
 			(font
@@
 	)
 	(label "AFE_OUTPUTS10"
-		(at 208.28 154.94 0)
+		(at 302.26 154.94 0)
 		(effects
 			(font
@@
 	)
 	(label "AFE_OUTPUTS21"
-		(at 208.28 172.72 0)
+		(at 208.28 152.4 0)
 		(effects
 			(font
@@
 	)
 	(label "AFE_OUTPUTS16"
-		(at 208.28 165.1 0)
+		(at 208.28 144.78 0)
 		(effects
 			(font
@@
 	)
 	(label "AFE_OUTPUTS6"
-		(at 269.24 147.32 180)
+		(at 363.22 147.32 180)
 		(effects
 			(font
@@
 	)
 	(label "AFE_OUTPUTS18"
-		(at 269.24 167.64 180)
+		(at 269.24 147.32 180)
 		(effects
 			(font
@@
 	)
 	(label "AFE_OUTPUTS31"
-		(at 361.95 149.86 180)
+		(at 363.22 170.18 180)
 		(effects
 			(font
@@
 	)
 	(label "AFE_OUTPUTS30"
-		(at 361.95 147.32 180)
+		(at 363.22 167.64 180)
 		(effects
 			(font
@@
 	)
 	(label "AFE_OUTPUTS42"
-		(at 361.95 167.64 180)
+		(at 269.24 167.64 180)
 		(effects
 			(font
@@
 	)
 	(label "AFE_OUTPUTS3"
-		(at 208.28 142.24 0)
+		(at 302.26 142.24 0)
 		(effects
 			(font
@@
 	)
 	(label "AFE_OUTPUTS34"
-		(at 303.53 154.94 0)
+		(at 302.26 175.26 0)
 		(effects
 			(font
@@
 	)
 	(label "AFE_OUTPUTS8"
-		(at 269.24 152.4 180)
+		(at 363.22 152.4 180)
 		(effects
 			(font
@@
 	)
 	(label "AFE_OUTPUTS36"
-		(at 361.95 157.48 180)
+		(at 269.24 157.48 180)
 		(effects
 			(font
@@
 	)
 	(label "AFE_OUTPUTS24"
-		(at 361.95 137.16 180)
+		(at 363.22 157.48 180)
 		(effects
 			(font
@@
 	)
 	(label "AFE_OUTPUTS27"
-		(at 303.53 142.24 0)
+		(at 302.26 162.56 0)
 		(effects
 			(font
@@
 	)
 	(label "AFE_OUTPUTS28"
-		(at 303.53 144.78 0)
+		(at 302.26 165.1 0)
 		(effects
 			(font
@@
 	)
 	(label "AFE_OUTPUTS32"
-		(at 361.95 152.4 180)
+		(at 363.22 172.72 180)
 		(effects
 			(font
@@
 	)
 	(label "AFE_OUTPUTS22"
-		(at 208.28 175.26 0)
+		(at 208.28 154.94 0)
 		(effects
 			(font
@@
 	)
 	(label "AFE_OUTPUTS13"
-		(at 269.24 160.02 180)
+		(at 269.24 139.7 180)
 		(effects
 			(font
@@
 	)
 	(label "AFE_OUTPUTS23"
-		(at 208.28 177.8 0)
+		(at 208.28 157.48 0)
 		(effects
 			(font
@@
 	)
 	(label "AFE_OUTPUTS44"
-		(at 361.95 172.72 180)
+		(at 269.24 172.72 180)
 		(effects
 			(font
@@
 	)
 	(label "AFE_OUTPUTS15"
-		(at 208.28 162.56 0)
+		(at 208.28 142.24 0)
 		(effects
 			(font
@@
 	)
 	(label "AFE_OUTPUTS4"
-		(at 208.28 144.78 0)
+		(at 302.26 144.78 0)
 		(effects
 			(font
@@
 	)
 	(hierarchical_label "USB_26MHZ"
-		(shape output)
+		(shape bidirectional)
 		(at 123.19 132.08 180)
 		(effects
@@
 			)
 		)
-		(property "Footprint" "Button_Switch_SMD:Nidec_Copal_CAS-120A"
+		(property "Footprint" "Button_Switch_SMD:SW_Push_SPST_NO_Alps_SKRK"
 			(at 147.32 215.9 0)
 			(hide yes)
